File: kicadProjects/0511/0511/0511.kicad_pcb (KiCad board)
At the start: 2 copper layers, 141 parts, among them SW1 SW_Push, SW10 SW_Push, SW11 SW_Push, SW12 SW_Push, SW13 SW_Push, SW14 SW_Push, SW15 SW_Push, SW16 SW_Push, SW17 SW_Push, SW18 SW_Push, SW19 SW_Push, SW2 SW_Push, SW20 SW_Push, SW21 SW_Push, SW22 SW_Push, SW23 SW_Push, SW24 SW_Push, SW25 SW_Push, SW26 SW_Push, SW27 SW_Push, SW28 SW_Push, SW29 SW_Push, SW3 SW_Push, SW30 SW_Push, SW31 SW_Push, SW32 SW_Push, SW4 SW_Push, SW5 SW_Push, SW6 SW_Push, SW7 SW_Push, SW8 SW_Push, SW9 SW_Push, U1 UDA1334A_Breakout, U2 YAAJ_BlackPill, U3 MCP23017, U4 MCP23017

Commit message: ajout connexions manquantes
Parts:
- added C34: C, Capacitor_THT:CP_Axial_L10.0mm_D4.5mm_P15.00mm_Horizontal, F.Cu at (-72.6, 195.8)
- added C35: C, Capacitor_THT:CP_Axial_L10.0mm_D4.5mm_P15.00mm_Horizontal, F.Cu at (-72.6, 212.9)
- added C36: C, Capacitor_THT:CP_Axial_L10.0mm_D4.5mm_P15.00mm_Horizontal, F.Cu at (-72.6, 204.4)
- added C37: C, Capacitor_THT:CP_Axial_L10.0mm_D4.5mm_P15.00mm_Horizontal, F.Cu at (-113.7, 168.0)
- added C38: C, Capacitor_THT:CP_Axial_L10.0mm_D4.5mm_P15.00mm_Horizontal, F.Cu at (-72.6, 84.4)
- added C39: C, Capacitor_THT:CP_Axial_L10.0mm_D4.5mm_P15.00mm_Horizontal, F.Cu at (-93.2, 140.1)
- added C40: C, Capacitor_THT:CP_Axial_L10.0mm_D4.5mm_P15.00mm_Horizontal, F.Cu at (-52.0, 84.4)
- added C41: C, Capacitor_THT:CP_Axial_L10.0mm_D4.5mm_P15.00mm_Horizontal, F.Cu at (-134.2, 140.1)
- added C42: C, Capacitor_THT:CP_Axial_L10.0mm_D4.5mm_P15.00mm_Horizontal, F.Cu at (-52.0, 140.1)
- added C43: C, Capacitor_THT:CP_Axial_L10.0mm_D4.5mm_P15.00mm_Horizontal, F.Cu at (-113.7, 84.4)
- added C44: C, Capacitor_THT:CP_Axial_L10.0mm_D4.5mm_P15.00mm_Horizontal, F.Cu at (-52.0, 112.2)
- added C45: C, Capacitor_THT:CP_Axial_L10.0mm_D4.5mm_P15.00mm_Horizontal, F.Cu at (-113.7, 140.1)
- added C46: C, Capacitor_THT:CP_Axial_L10.0mm_D4.5mm_P15.00mm_Horizontal, F.Cu at (-93.2, 195.8)
- added C47: C, Capacitor_THT:CP_Axial_L10.0mm_D4.5mm_P15.00mm_Horizontal, F.Cu at (-157.8, 123.5)
- added C48: C, Capacitor_THT:CP_Axial_L10.0mm_D4.5mm_P15.00mm_Horizontal, F.Cu at (-72.6, 112.2)
- added C49: C, Capacitor_THT:CP_Axial_L10.0mm_D4.5mm_P15.00mm_Horizontal, F.Cu at (-113.7, 56.5)
- added C50: C, Capacitor_THT:CP_Axial_L10.0mm_D4.5mm_P15.00mm_Horizontal, F.Cu at (-31.5, 140.1)
- added C51: C, Capacitor_THT:CP_Axial_L10.0mm_D4.5mm_P15.00mm_Horizontal, F.Cu at (-31.5, 56.5)
- added C52: C, Capacitor_THT:CP_Axial_L10.0mm_D4.5mm_P15.00mm_Horizontal, F.Cu at (-93.2, 56.5)
- added C53: C, Capacitor_THT:CP_Axial_L10.0mm_D4.5mm_P15.00mm_Horizontal, F.Cu at (-31.5, 112.2)
- added C54: C, Capacitor_THT:CP_Axial_L10.0mm_D4.5mm_P15.00mm_Horizontal, F.Cu at (-134.2, 195.8)
- added C55: C, Capacitor_THT:CP_Axial_L10.0mm_D4.5mm_P15.00mm_Horizontal, F.Cu at (-134.2, 112.2)
- added C56: C, Capacitor_THT:CP_Axial_L10.0mm_D4.5mm_P15.00mm_Horizontal, F.Cu at (-134.2, 84.4)
- added C57: C, Capacitor_THT:CP_Axial_L10.0mm_D4.5mm_P15.00mm_Horizontal, F.Cu at (-134.2, 56.5)
- added C58: C, Capacitor_THT:CP_Axial_L10.0mm_D4.5mm_P15.00mm_Horizontal, F.Cu at (-72.6, 168.0)
- added C59: C, Capacitor_THT:CP_Axial_L10.0mm_D4.5mm_P15.00mm_Horizontal, F.Cu at (-72.6, 56.5)
- added C60: C, Capacitor_THT:CP_Axial_L10.0mm_D4.5mm_P15.00mm_Horizontal, F.Cu at (-52.0, 56.5)
- added C61: C, Capacitor_THT:CP_Axial_L10.0mm_D4.5mm_P15.00mm_Horizontal, F.Cu at (-72.6, 140.1)
- added C62: C, Capacitor_THT:CP_Axial_L10.0mm_D4.5mm_P15.00mm_Horizontal, F.Cu at (-93.2, 112.2)
- added C63: C, Capacitor_THT:CP_Axial_L10.0mm_D4.5mm_P15.00mm_Horizontal, F.Cu at (-113.7, 195.8)
- added C64: C, Capacitor_THT:CP_Axial_L10.0mm_D4.5mm_P15.00mm_Horizontal, F.Cu at (-157.8, 151.4)
- added C65: C, Capacitor_THT:CP_Axial_L10.0mm_D4.5mm_P15.00mm_Horizontal, F.Cu at (-157.8, 95.6)
- added C66: C, Capacitor_THT:CP_Axial_L10.0mm_D4.5mm_P15.00mm_Horizontal, F.Cu at (-93.2, 168.0)
- added C67: C, Capacitor_THT:CP_Axial_L10.0mm_D4.5mm_P15.00mm_Horizontal, F.Cu at (-93.2, 84.4)
- added C68: C, Capacitor_THT:CP_Axial_L10.0mm_D4.5mm_P15.00mm_Horizontal, F.Cu at (-157.8, 179.2)
- added C69: C, Capacitor_THT:CP_Axial_L10.0mm_D4.5mm_P15.00mm_Horizontal, F.Cu at (-31.5, 84.4)
- added C70: C, Capacitor_THT:CP_Axial_L10.0mm_D4.5mm_P15.00mm_Horizontal, F.Cu at (-113.7, 112.2)
- added C71: C, Capacitor_THT:CP_Axial_L10.0mm_D4.5mm_P15.00mm_Horizontal, F.Cu at (-134.2, 168.0)
- added D33: LED, Diode_THT:D_DO-41_SOD81_P10.16mm_Horizontal, F.Cu at (-113.6, 188.2)
- added D34: LED, Diode_THT:D_DO-41_SOD81_P10.16mm_Horizontal, F.Cu at (-72.5, 104.6)
- added D35: LED, Diode_THT:D_DO-41_SOD81_P10.16mm_Horizontal, F.Cu at (-93.0, 160.3)
- added D36: LED, Diode_THT:D_DO-41_SOD81_P10.16mm_Horizontal, F.Cu at (-52.0, 104.6)
- added D37: LED, Diode_THT:D_DO-41_SOD81_P10.16mm_Horizontal, F.Cu at (-134.2, 160.3)
- added D38: LED, Diode_THT:D_DO-41_SOD81_P10.16mm_Horizontal, F.Cu at (-52.0, 160.3)
- added D39: LED, Diode_THT:D_DO-41_SOD81_P10.16mm_Horizontal, F.Cu at (-113.6, 104.6)
- added D40: LED, Diode_THT:D_DO-41_SOD81_P10.16mm_Horizontal, F.Cu at (-52.0, 132.5)
- added D41: LED, Diode_THT:D_DO-41_SOD81_P10.16mm_Horizontal, F.Cu at (-113.6, 160.3)
- added D42: LED, Diode_THT:D_DO-41_SOD81_P10.16mm_Horizontal, F.Cu at (-93.0, 216.1)
- added D43: LED, Diode_THT:D_DO-41_SOD81_P10.16mm_Horizontal, F.Cu at (-157.7, 143.7)
- added D44: LED, Diode_THT:D_DO-41_SOD81_P10.16mm_Horizontal, F.Cu at (-72.5, 132.5)
- added D45: LED, Diode_THT:D_DO-41_SOD81_P10.16mm_Horizontal, F.Cu at (-113.6, 76.7)
- added D46: LED, Diode_THT:D_DO-41_SOD81_P10.16mm_Horizontal, F.Cu at (-31.4, 160.3)
- added D47: LED, Diode_THT:D_DO-41_SOD81_P10.16mm_Horizontal, F.Cu at (-31.4, 76.7)
- added D48: LED, Diode_THT:D_DO-41_SOD81_P10.16mm_Horizontal, F.Cu at (-93.0, 76.7)
- added D49: LED, Diode_THT:D_DO-41_SOD81_P10.16mm_Horizontal, F.Cu at (-31.4, 132.5)
- added D50: LED, Diode_THT:D_DO-41_SOD81_P10.16mm_Horizontal, F.Cu at (-134.2, 216.1)
- added D51: LED, Diode_THT:D_DO-41_SOD81_P10.16mm_Horizontal, F.Cu at (-134.2, 132.5)
- added D52: LED, Diode_THT:D_DO-41_SOD81_P10.16mm_Horizontal, F.Cu at (-134.2, 104.6)
- added D53: LED, Diode_THT:D_DO-41_SOD81_P10.16mm_Horizontal, F.Cu at (-134.2, 76.7)
- added D54: LED, Diode_THT:D_DO-41_SOD81_P10.16mm_Horizontal, F.Cu at (-72.5, 188.2)
- added D55: LED, Diode_THT:D_DO-41_SOD81_P10.16mm_Horizontal, F.Cu at (-72.5, 76.7)
- added D56: LED, Diode_THT:D_DO-41_SOD81_P10.16mm_Horizontal, F.Cu at (-52.0, 76.7)
- added D57: LED, Diode_THT:D_DO-41_SOD81_P10.16mm_Horizontal, F.Cu at (-72.5, 160.3)
- added D58: LED, Diode_THT:D_DO-41_SOD81_P10.16mm_Horizontal, F.Cu at (-93.0, 132.5)
- added D59: LED, Diode_THT:D_DO-41_SOD81_P10.16mm_Horizontal, F.Cu at (-113.6, 216.1)
- added D60: LED, Diode_THT:D_DO-41_SOD81_P10.16mm_Horizontal, F.Cu at (-157.7, 171.6)
- added D61: LED, Diode_THT:D_DO-41_SOD81_P10.16mm_Horizontal, F.Cu at (-157.7, 115.9)
- added D62: LED, Diode_THT:D_DO-41_SOD81_P10.16mm_Horizontal, F.Cu at (-93.0, 188.2)
- added D63: LED, Diode_THT:D_DO-41_SOD81_P10.16mm_Horizontal, F.Cu at (-93.0, 104.6)
- added D64: LED, Diode_THT:D_DO-41_SOD81_P10.16mm_Horizontal, F.Cu at (-157.7, 199.5)
- added D65: LED, Diode_THT:D_DO-41_SOD81_P10.16mm_Horizontal, F.Cu at (-31.4, 104.6)
- added D66: LED, Diode_THT:D_DO-41_SOD81_P10.16mm_Horizontal, F.Cu at (-113.6, 132.5)
- added D67: LED, Diode_THT:D_DO-41_SOD81_P10.16mm_Horizontal, F.Cu at (-134.2, 188.2)
- added R41: R, Resistor_SMD:R_0603_1608Metric, F.Cu at (-99.6, 187.3)
- added R42: R, Resistor_SMD:R_0603_1608Metric, F.Cu at (-58.5, 103.7)
- added R43: R, Resistor_SMD:R_0603_1608Metric, F.Cu at (-79.0, 159.5)
- added R44: R, Resistor_SMD:R_0603_1608Metric, F.Cu at (-37.9, 103.7)
- added R45: R, Resistor_SMD:R_0603_1608Metric, F.Cu at (-120.1, 159.5)
- added R46: R, Resistor_SMD:R_0603_1608Metric, F.Cu at (-37.9, 159.5)
- added R47: R, Resistor_SMD:R_0603_1608Metric, F.Cu at (-99.6, 103.7)
- added R48: R, Resistor_SMD:R_0603_1608Metric, F.Cu at (-37.9, 131.6)
- added R49: R, Resistor_SMD:R_0603_1608Metric, F.Cu at (-99.6, 159.5)
- added R50: R, Resistor_SMD:R_0603_1608Metric, F.Cu at (-79.0, 215.2)
- added R51: R, Resistor_SMD:R_0603_1608Metric, F.Cu at (-143.7, 142.9)
- added R52: R, Resistor_SMD:R_0603_1608Metric, F.Cu at (-58.5, 131.6)
- added R53: R, Resistor_SMD:R_0603_1608Metric, F.Cu at (-99.6, 75.9)
- added R54: R, Resistor_SMD:R_0603_1608Metric, F.Cu at (-17.4, 159.5)
- added R55: R, Resistor_SMD:R_0603_1608Metric, F.Cu at (-17.4, 75.9)
- added R56: R, Resistor_SMD:R_0603_1608Metric, F.Cu at (-79.0, 75.9)
- added R57: R, Resistor_SMD:R_0603_1608Metric, F.Cu at (-17.4, 131.6)
- added R58: R, Resistor_SMD:R_0603_1608Metric, F.Cu at (-120.1, 215.2)
- added R59: R, Resistor_SMD:R_0603_1608Metric, F.Cu at (-120.1, 131.6)
- added R60: R, Resistor_SMD:R_0603_1608Metric, F.Cu at (-120.1, 103.7)
- added R61: R, Resistor_SMD:R_0603_1608Metric, F.Cu at (-120.1, 75.9)
- added R62: R, Resistor_SMD:R_0603_1608Metric, F.Cu at (-58.5, 187.3)
- added R63: R, Resistor_SMD:R_0603_1608Metric, F.Cu at (-58.5, 75.9)
- added R64: R, Resistor_SMD:R_0603_1608Metric, F.Cu at (-37.9, 75.9)
- added R65: R, Resistor_SMD:R_0603_1608Metric, F.Cu at (-58.5, 159.5)
- added R66: R, Resistor_SMD:R_0603_1608Metric, F.Cu at (-79.0, 131.6)
- added R67: R, Resistor_SMD:R_0603_1608Metric, F.Cu at (-99.6, 215.2)
- added R68: R, Resistor_SMD:R_0603_1608Metric, F.Cu at (-143.7, 170.7)
- added R69: R, Resistor_SMD:R_0603_1608Metric, F.Cu at (-143.7, 115.0)
- added R70: R, Resistor_SMD:R_0603_1608Metric, F.Cu at (-79.0, 187.3)
- added R71: R, Resistor_SMD:R_0603_1608Metric, F.Cu at (-79.0, 103.7)
- added R72: R, Resistor_SMD:R_0603_1608Metric, F.Cu at (-143.7, 198.6)
- added R73: R, Resistor_SMD:R_0603_1608Metric, F.Cu at (-17.4, 103.7)
- added R74: R, Resistor_SMD:R_0603_1608Metric, F.Cu at (-99.6, 131.6)
- added R75: R, Resistor_SMD:R_0603_1608Metric, F.Cu at (-120.1, 187.3)
- added SW33: SW_Push, Button_Switch_Keyboard:SW_Cherry_MX_1.00u_PCB, F.Cu at (-105.4, 173.5)
- added SW34: SW_Push, Button_Switch_Keyboard:SW_Cherry_MX_1.00u_PCB, F.Cu at (-64.3, 89.9)
- added SW35: SW_Push, Button_Switch_Keyboard:SW_Cherry_MX_1.00u_PCB, F.Cu at (-84.8, 145.6)
- added SW36: SW_Push, Button_Switch_Keyboard:SW_Cherry_MX_1.00u_PCB, F.Cu at (-43.7, 89.9)
- added SW37: SW_Push, Button_Switch_Keyboard:SW_Cherry_MX_1.00u_PCB, F.Cu at (-125.9, 145.6)
- added SW38: SW_Push, Button_Switch_Keyboard:SW_Cherry_MX_1.00u_PCB, F.Cu at (-43.7, 145.6)
- added SW39: SW_Push, Button_Switch_Keyboard:SW_Cherry_MX_1.00u_PCB, F.Cu at (-105.4, 89.9)
- added SW40: SW_Push, Button_Switch_Keyboard:SW_Cherry_MX_1.00u_PCB, F.Cu at (-43.7, 117.7)
- added SW41: SW_Push, Button_Switch_Keyboard:SW_Cherry_MX_1.00u_PCB, F.Cu at (-105.4, 145.6)
- added SW42: SW_Push, Button_Switch_Keyboard:SW_Cherry_MX_1.00u_PCB, F.Cu at (-84.8, 201.3)
- added SW43: SW_Push, Button_Switch_Keyboard:SW_Cherry_MX_1.00u_PCB, F.Cu at (-149.5, 129.0)
- added SW44: SW_Push, Button_Switch_Keyboard:SW_Cherry_MX_1.00u_PCB, F.Cu at (-64.3, 117.7)
- added SW45: SW_Push, Button_Switch_Keyboard:SW_Cherry_MX_1.00u_PCB, F.Cu at (-105.4, 62.0)
- added SW46: SW_Push, Button_Switch_Keyboard:SW_Cherry_MX_1.00u_PCB, F.Cu at (-23.2, 145.6)
- added SW47: SW_Push, Button_Switch_Keyboard:SW_Cherry_MX_1.00u_PCB, F.Cu at (-23.2, 62.0)
- added SW48: SW_Push, Button_Switch_Keyboard:SW_Cherry_MX_1.00u_PCB, F.Cu at (-84.8, 62.0)
- added SW49: SW_Push, Button_Switch_Keyboard:SW_Cherry_MX_1.00u_PCB, F.Cu at (-23.2, 117.7)
- added SW50: SW_Push, Button_Switch_Keyboard:SW_Cherry_MX_1.00u_PCB, F.Cu at (-125.9, 201.3)
- added SW51: SW_Push, Button_Switch_Keyboard:SW_Cherry_MX_1.00u_PCB, F.Cu at (-125.9, 117.7)
- added SW52: SW_Push, Button_Switch_Keyboard:SW_Cherry_MX_1.00u_PCB, F.Cu at (-125.9, 89.9)
- added SW53: SW_Push, Button_Switch_Keyboard:SW_Cherry_MX_1.00u_PCB, F.Cu at (-125.9, 62.0)
- added SW54: SW_Push, Button_Switch_Keyboard:SW_Cherry_MX_1.00u_PCB, F.Cu at (-64.3, 173.5)
- added SW55: SW_Push, Button_Switch_Keyboard:SW_Cherry_MX_1.00u_PCB, F.Cu at (-64.3, 62.0)
- added SW56: SW_Push, Button_Switch_Keyboard:SW_Cherry_MX_1.00u_PCB, F.Cu at (-43.7, 62.0)
- added SW57: SW_Push, Button_Switch_Keyboard:SW_Cherry_MX_1.00u_PCB, F.Cu at (-64.3, 145.6)
- added SW58: SW_Push, Button_Switch_Keyboard:SW_Cherry_MX_1.00u_PCB, F.Cu at (-84.8, 117.7)
- added SW59: SW_Push, Button_Switch_Keyboard:SW_Cherry_MX_1.00u_PCB, F.Cu at (-105.4, 201.3)
- added SW60: SW_Push, Button_Switch_Keyboard:SW_Cherry_MX_1.00u_PCB, F.Cu at (-149.5, 156.9)
- added SW61: SW_Push, Button_Switch_Keyboard:SW_Cherry_MX_1.00u_PCB, F.Cu at (-149.5, 101.1)
- added SW62: SW_Push, Button_Switch_Keyboard:SW_Cherry_MX_1.00u_PCB, F.Cu at (-84.8, 173.5)
- added SW63: SW_Push, Button_Switch_Keyboard:SW_Cherry_MX_1.00u_PCB, F.Cu at (-84.8, 89.9)
- added SW64: SW_Push, Button_Switch_Keyboard:SW_Cherry_MX_1.00u_PCB, F.Cu at (-149.5, 184.7)
- added SW65: SW_Push, Button_Switch_Keyboard:SW_Cherry_MX_1.00u_PCB, F.Cu at (-23.2, 89.9)
- added SW66: SW_Push, Button_Switch_Keyboard:SW_Cherry_MX_1.00u_PCB, F.Cu at (-105.4, 117.7)
- added SW67: SW_Push, Button_Switch_Keyboard:SW_Cherry_MX_1.00u_PCB, F.Cu at (-125.9, 173.5)
- added U5: MCP23017, Package_DIP:DIP-28_W7.62mm, F.Cu at (-158.0, 55.0)
- added U6: MCP23017, Package_DIP:DIP-28_W7.62mm, F.Cu at (-147.2, 55.0)
- R1: value R_Variable -> R; footprint Button_Switch_THT:Push_E-Switch_KS01Q01 -> Resistor_SMD:R_0603_1608Metric
- R2: value ~ -> R_Variable; footprint Resistor_THT:R_Axial_DIN0207_L6.3mm_D2.5mm_P7.62mm_Horizontal -> Button_Switch_THT:Push_E-Switch_KS01Q01
- R3: value R -> ~; footprint Resistor_SMD:R_0603_1608Metric -> Resistor_THT:R_Axial_DIN0207_L6.3mm_D2.5mm_P7.62mm_Horizontal
Connections:
- C10 pad 1: /Button_RCD8/To_MCP_PIN -> /Button_RCD75/To_MCP_PIN
- C11 pad 1: /Button_RCD9/To_MCP_PIN -> /Button_RCD76/To_MCP_PIN
- C12 pad 1: /Button_RCD10/To_MCP_PIN -> /Button_RCD64/To_MCP_PIN
- C13 pad 1: /Button_RCD11/To_MCP_PIN -> /Button_RCD65/To_MCP_PIN
- C14 pad 1: /Button_RCD12/To_MCP_PIN -> /Button_RCD66/To_MCP_PIN
- C15 pad 1: /Button_RCD13/To_MCP_PIN -> /Button_RCD67/To_MCP_PIN
- C16 pad 1: /Button_RCD14/To_MCP_PIN -> /Button_RCD68/To_MCP_PIN
- C17 pad 1: /Button_RCD15/To_MCP_PIN -> /Button_RCD69/To_MCP_PIN
- C18 pad 1: /Button_RCD16/To_MCP_PIN -> /Button_RCD70/To_MCP_PIN
- C19 pad 1: /Button_RCD17/To_MCP_PIN -> /Button_RCD81/To_MCP_PIN
- C2 pad 1: /Button_RCD/To_MCP_PIN -> +3.3V
- C20 pad 1: /Button_RCD18/To_MCP_PIN -> /Button_RCD79/To_MCP_PIN
- C21 pad 1: /Button_RCD19/To_MCP_PIN -> /Button_RCD16/To_MCP_PIN
- C22 pad 1: /Button_RCD20/To_MCP_PIN -> /Button_RCD17/To_MCP_PIN
- C23 pad 1: /Button_RCD21/To_MCP_PIN -> /Button_RCD18/To_MCP_PIN
- C24 pad 1: /Button_RCD22/To_MCP_PIN -> /Button_RCD80/To_MCP_PIN
- C25 pad 1: /Button_RCD23/To_MCP_PIN -> /Button_RCD20/To_MCP_PIN
- C26 pad 1: /Button_RCD24/To_MCP_PIN -> /Button_RCD21/To_MCP_PIN
- C27 pad 1: /Button_RCD25/To_MCP_PIN -> /Button_RCD22/To_MCP_PIN
- C28 pad 1: /Button_RCD26/To_MCP_PIN -> /Button_RCD23/To_MCP_PIN
- C29 pad 1: /Button_RCD27/To_MCP_PIN -> /Button_RCD24/To_MCP_PIN
- C3 pad 1: /Button_RCD1/To_MCP_PIN -> +3.3V
- C30 pad 1: /Button_RCD28/To_MCP_PIN -> /Button_RCD25/To_MCP_PIN
- C31 pad 1: /Button_RCD29/To_MCP_PIN -> /Button_RCD26/To_MCP_PIN
- C32 pad 1: /Button_RCD30/To_MCP_PIN -> /Button_RCD27/To_MCP_PIN
- C33 pad 1: /Button_RCD31/To_MCP_PIN -> /Button_RCD28/To_MCP_PIN
- C4 pad 1: /Button_RCD2/To_MCP_PIN -> +3.3V
- C5 pad 1: /Button_RCD3/To_MCP_PIN -> /Button_RCD19/To_MCP_PIN
- C6 pad 1: /Button_RCD4/To_MCP_PIN -> /Button_RCD71/To_MCP_PIN
- C7 pad 1: /Button_RCD5/To_MCP_PIN -> /Button_RCD72/To_MCP_PIN
- C8 pad 1: /Button_RCD6/To_MCP_PIN -> /Button_RCD73/To_MCP_PIN
- C9 pad 1: /Button_RCD7/To_MCP_PIN -> /Button_RCD74/To_MCP_PIN
- D1 pad 1: /Button_RCD/To_MCP_PIN -> /Button_RCD19/To_MCP_PIN
- D10 pad 1: /Button_RCD9/To_MCP_PIN -> /Button_RCD66/To_MCP_PIN
- D11 pad 1: /Button_RCD10/To_MCP_PIN -> /Button_RCD67/To_MCP_PIN
- D12 pad 1: /Button_RCD11/To_MCP_PIN -> /Button_RCD68/To_MCP_PIN
- D13 pad 1: /Button_RCD12/To_MCP_PIN -> /Button_RCD69/To_MCP_PIN
- D14 pad 1: /Button_RCD13/To_MCP_PIN -> /Button_RCD70/To_MCP_PIN
- D15 pad 1: /Button_RCD14/To_MCP_PIN -> /Button_RCD81/To_MCP_PIN
- D16 pad 1: /Button_RCD15/To_MCP_PIN -> /Button_RCD79/To_MCP_PIN
- D2 pad 1: /Button_RCD1/To_MCP_PIN -> /Button_RCD71/To_MCP_PIN
- D20 pad 1: /Button_RCD19/To_MCP_PIN -> /Button_RCD80/To_MCP_PIN
- D3 pad 1: /Button_RCD2/To_MCP_PIN -> /Button_RCD72/To_MCP_PIN
- D4 pad 1: /Button_RCD3/To_MCP_PIN -> /Button_RCD73/To_MCP_PIN
- D5 pad 1: /Button_RCD4/To_MCP_PIN -> /Button_RCD74/To_MCP_PIN
- D6 pad 1: /Button_RCD5/To_MCP_PIN -> /Button_RCD75/To_MCP_PIN
- D7 pad 1: /Button_RCD6/To_MCP_PIN -> /Button_RCD76/To_MCP_PIN
- D8 pad 1: /Button_RCD7/To_MCP_PIN -> /Button_RCD64/To_MCP_PIN
- D9 pad 1: /Button_RCD8/To_MCP_PIN -> /Button_RCD65/To_MCP_PIN
- R1 pad 1: Net-(U1-3V) -> +3.3V
- R1 pad 2: Net-(U2-PA1) -> Net-(U3-~{RESET})
- R10 pad 1: /Button_RCD1/To_MCP_PIN -> /Button_RCD71/To_MCP_PIN
- R11 pad 1: /Button_RCD2/To_MCP_PIN -> /Button_RCD72/To_MCP_PIN
- R12 pad 1: /Button_RCD3/To_MCP_PIN -> /Button_RCD73/To_MCP_PIN
- R13 pad 1: /Button_RCD4/To_MCP_PIN -> /Button_RCD74/To_MCP_PIN
- R14 pad 1: /Button_RCD5/To_MCP_PIN -> /Button_RCD75/To_MCP_PIN
- R15 pad 1: /Button_RCD6/To_MCP_PIN -> /Button_RCD76/To_MCP_PIN
- R16 pad 1: /Button_RCD7/To_MCP_PIN -> /Button_RCD64/To_MCP_PIN
- R17 pad 1: /Button_RCD8/To_MCP_PIN -> /Button_RCD65/To_MCP_PIN
- R18 pad 1: /Button_RCD9/To_MCP_PIN -> /Button_RCD66/To_MCP_PIN
- R19 pad 1: /Button_RCD10/To_MCP_PIN -> /Button_RCD67/To_MCP_PIN
- R2 pad 1: Net-(U2-PA1) -> +3.3V
- R2 pad 2: Net-(R2-Pad2) -> Net-(U2-PA1)
- R20 pad 1: /Button_RCD11/To_MCP_PIN -> /Button_RCD68/To_MCP_PIN
- R21 pad 1: /Button_RCD12/To_MCP_PIN -> /Button_RCD69/To_MCP_PIN
- R22 pad 1: /Button_RCD13/To_MCP_PIN -> /Button_RCD70/To_MCP_PIN
- R23 pad 1: /Button_RCD14/To_MCP_PIN -> /Button_RCD81/To_MCP_PIN
- R24 pad 1: /Button_RCD15/To_MCP_PIN -> /Button_RCD79/To_MCP_PIN
- R28 pad 1: /Button_RCD19/To_MCP_PIN -> /Button_RCD80/To_MCP_PIN
- R3 pad 1: +3.3V -> Net-(U2-PA1)
- R3 pad 2: Net-(U2-PB8) -> GND
- R4 pad 2: Net-(U2-PB9) -> Net-(U4-~{RESET})
- R5 pad 2: Net-(U3-~{RESET}) -> Net-(U2-PB8)
- R6 pad 2: Net-(U2-PB8) -> Net-(U2-PB9)
- R7 pad 2: Net-(U4-~{RESET}) -> Net-(U5-~{RESET})
- R8 pad 2: Net-(U2-PB9) -> Net-(U6-~{RESET})
- R9 pad 1: /Button_RCD/To_MCP_PIN -> /Button_RCD19/To_MCP_PIN
- SW1 pad 2: /Button_RCD/To_MCP_PIN -> /Button_RCD19/To_MCP_PIN
- SW10 pad 2: /Button_RCD9/To_MCP_PIN -> /Button_RCD66/To_MCP_PIN
- SW11 pad 2: /Button_RCD10/To_MCP_PIN -> /Button_RCD67/To_MCP_PIN
- SW12 pad 2: /Button_RCD11/To_MCP_PIN -> /Button_RCD68/To_MCP_PIN
- SW13 pad 2: /Button_RCD12/To_MCP_PIN -> /Button_RCD69/To_MCP_PIN
- SW14 pad 2: /Button_RCD13/To_MCP_PIN -> /Button_RCD70/To_MCP_PIN
- SW15 pad 2: /Button_RCD14/To_MCP_PIN -> /Button_RCD81/To_MCP_PIN
- SW16 pad 2: /Button_RCD15/To_MCP_PIN -> /Button_RCD79/To_MCP_PIN
- SW2 pad 2: /Button_RCD1/To_MCP_PIN -> /Button_RCD71/To_MCP_PIN
- SW20 pad 2: /Button_RCD19/To_MCP_PIN -> /Button_RCD80/To_MCP_PIN
- SW3 pad 2: /Button_RCD2/To_MCP_PIN -> /Button_RCD72/To_MCP_PIN
- SW4 pad 2: /Button_RCD3/To_MCP_PIN -> /Button_RCD73/To_MCP_PIN
- SW5 pad 2: /Button_RCD4/To_MCP_PIN -> /Button_RCD74/To_MCP_PIN
- SW6 pad 2: /Button_RCD5/To_MCP_PIN -> /Button_RCD75/To_MCP_PIN
- SW7 pad 2: /Button_RCD6/To_MCP_PIN -> /Button_RCD76/To_MCP_PIN
- SW8 pad 2: /Button_RCD7/To_MCP_PIN -> /Button_RCD64/To_MCP_PIN
- SW9 pad 2: /Button_RCD8/To_MCP_PIN -> /Button_RCD65/To_MCP_PIN
- U1 pad 1: unconnected-(U1-VIN-Pad1) -> +3.3V
- U1 pad 2: Net-(U1-3V) -> unconnected-(U1-3V-Pad2)
- U1 pad 3: unconnected-(U1-GND-Pad3) -> GND
- U2 pad 1: unconnected-(U2-PB12-Pad1) -> Net-(U2-PA10)
- U2 pad 16: Net-(U1-3V) -> unconnected-(U2-3V3-Pad16)
- U2 pad 17: Net-(R2-Pad2) -> GND
- U2 pad 18: Net-(R2-Pad2) -> GND
- U2 pad 2: unconnected-(U2-PB13-Pad2) -> Net-(U2-PA10)
- U2 pad 3: unconnected-(U2-PB14-Pad3) -> Net-(U2-PA10)
- U2 pad 4: unconnected-(U2-PB15-Pad4) -> Net-(U2-PA10)
- U2 pad 5: unconnected-(U2-PA8-Pad5) -> Net-(U2-PA10)
- U2 pad 7: unconnected-(U2-PA10-Pad7) -> Net-(U2-PA10)
- U3 pad 1: /Button_RCD13/To_MCP_PIN -> /Button_RCD61/To_MCP_PIN
- U3 pad 15: GND -> +3.3V
- U3 pad 16: GND -> +3.3V
- U3 pad 2: /Button_RCD12/To_MCP_PIN -> /Button_RCD60/To_MCP_PIN
- U3 pad 20: unconnected-(U3-INTA-Pad20) -> Net-(U2-PA10)
- U3 pad 21: /Button_RCD6/To_MCP_PIN -> /Button_RCD52/To_MCP_PIN
- U3 pad 22: /Button_RCD5/To_MCP_PIN -> /Button_RCD51/To_MCP_PIN
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
Commit message: overriden pcb file
Parts:
- moved C65 373.7 mm to (213.1, 141.1)
- moved D61 373.7 mm to (213.2, 161.4)
- moved R69 373.7 mm to (227.2, 160.5)
- moved SW61 373.7 mm to (221.4, 146.6)
- moved C55 351.6 mm to (213.1, 57.5)
- moved D51 351.6 mm to (213.2, 77.8)
- moved SW51 351.6 mm to (221.4, 63.0)
- moved R59 351.6 mm to (227.2, 76.9)
- moved C71 347.3 mm to (213.1, 169.0)
- moved D67 347.3 mm to (213.2, 189.2)
- moved SW67 347.3 mm to (221.4, 174.5)
- moved R75 347.3 mm to (227.2, 188.4)
- moved C36 339.6 mm to (233.6, 57.5)
- moved D42 337.1 mm to (233.7, 133.5)
- moved R50 337.1 mm to (247.8, 132.6)
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
Commit message: adaptation empreintes mcp23017 ajout valeurs aux résistances corrections empreintes des résistances et condensateurs
Parts:
- added R100: 150R, Resistor_SMD:R_0603_1608Metric, F.Cu at (312.9, 71.5)
- added R101: 10K, Resistor_SMD:R_0603_1608Metric, F.Cu at (325.6, 33.9)
- added R102: 150R, Resistor_SMD:R_0603_1608Metric, F.Cu at (325.6, 36.4)
- added R103: 10K, Resistor_SMD:R_0603_1608Metric, F.Cu at (306.5, 33.9)
- added R104: 150R, Resistor_SMD:R_0603_1608Metric, F.Cu at (306.5, 36.4)
- added R105: 10K, Resistor_SMD:R_0603_1608Metric, F.Cu at (306.5, 62.0)
- added R106: 150R, Resistor_SMD:R_0603_1608Metric, F.Cu at (306.5, 64.5)
- added R107: 10K, Resistor_SMD:R_0603_1608Metric, F.Cu at (300.2, 62.0)
- added R108: 150R, Resistor_SMD:R_0603_1608Metric, F.Cu at (300.2, 64.5)
- added R109: 10K, Resistor_SMD:R_0603_1608Metric, F.Cu at (300.2, 55.0)
- added R110: 150R, Resistor_SMD:R_0603_1608Metric, F.Cu at (300.2, 57.5)
- added R111: 10K, Resistor_SMD:R_0603_1608Metric, F.Cu at (300.2, 40.9)
- added R112: 150R, Resistor_SMD:R_0603_1608Metric, F.Cu at (300.2, 43.4)
- added R113: 10K, Resistor_SMD:R_0603_1608Metric, F.Cu at (290.1, 63.6)
- added R114: 150R, Resistor_SMD:R_0603_1608Metric, F.Cu at (290.1, 66.1)
- added R115: 10K, Resistor_SMD:R_0603_1608Metric, F.Cu at (319.2, 62.0)
- added R116: 150R, Resistor_SMD:R_0603_1608Metric, F.Cu at (319.2, 64.5)
- added R117: 10K, Resistor_SMD:R_0603_1608Metric, F.Cu at (312.9, 33.9)
- added R118: 150R, Resistor_SMD:R_0603_1608Metric, F.Cu at (312.9, 36.4)
- added R119: 10K, Resistor_SMD:R_0603_1608Metric, F.Cu at (319.2, 33.9)
- added R120: 150R, Resistor_SMD:R_0603_1608Metric, F.Cu at (319.2, 36.4)
- added R121: 10K, Resistor_SMD:R_0603_1608Metric, F.Cu at (325.6, 55.0)
- added R122: 150R, Resistor_SMD:R_0603_1608Metric, F.Cu at (325.6, 57.5)
- added R123: 10K, Resistor_SMD:R_0603_1608Metric, F.Cu at (319.2, 47.9)
- added R124: 150R, Resistor_SMD:R_0603_1608Metric, F.Cu at (319.2, 50.5)
- added R125: 10K, Resistor_SMD:R_0603_1608Metric, F.Cu at (312.9, 47.9)
- added R126: 150R, Resistor_SMD:R_0603_1608Metric, F.Cu at (312.9, 50.5)
- added R127: 10K, Resistor_SMD:R_0603_1608Metric, F.Cu at (290.1, 56.6)
- added R128: 150R, Resistor_SMD:R_0603_1608Metric, F.Cu at (290.1, 59.1)
- added R129: 10K, Resistor_SMD:R_0603_1608Metric, F.Cu at (325.6, 62.0)
- added R130: 150R, Resistor_SMD:R_0603_1608Metric, F.Cu at (325.6, 64.5)
- added R131: 10K, Resistor_SMD:R_0603_1608Metric, F.Cu at (312.9, 55.0)
- added R132: 150R, Resistor_SMD:R_0603_1608Metric, F.Cu at (312.9, 57.5)
- added R133: 10K, Resistor_SMD:R_0603_1608Metric, F.Cu at (312.9, 40.9)
- added R134: 150R, Resistor_SMD:R_0603_1608Metric, F.Cu at (312.9, 43.4)
- added R135: 10K, Resistor_SMD:R_0603_1608Metric, F.Cu at (283.7, 63.6)
- added R136: 150R, Resistor_SMD:R_0603_1608Metric, F.Cu at (283.7, 66.1)
- added R137: 10K, Resistor_SMD:R_0603_1608Metric, F.Cu at (300.2, 47.9)
- added R138: 150R, Resistor_SMD:R_0603_1608Metric, F.Cu at (300.2, 50.5)
- added R139: 10K, Resistor_SMD:R_0603_1608Metric, F.Cu at (300.2, 69.0)
- added R140: 150R, Resistor_SMD:R_0603_1608Metric, F.Cu at (300.2, 71.5)
- added R141: 10K, Resistor_SMD:R_0603_1608Metric, F.Cu at (319.2, 40.9)
- added R142: 150R, Resistor_SMD:R_0603_1608Metric, F.Cu at (319.2, 43.4)
- added R143: 10K, Resistor_SMD:R_0603_1608Metric, F.Cu at (12.2, 31.5)
- added R144: 150R, Resistor_SMD:R_0603_1608Metric, F.Cu at (12.2, 34.0)
- added R145: 10K, Resistor_SMD:R_0603_1608Metric, F.Cu at (18.2, 31.5)
- added R146: 150R, Resistor_SMD:R_0603_1608Metric, F.Cu at (18.2, 34.0)
- added R147: 10K, Resistor_SMD:R_0603_1608Metric, F.Cu at (12.2, 38.5)
- added R148: 150R, Resistor_SMD:R_0603_1608Metric, F.Cu at (12.2, 41.0)
- added R149: 10K, Resistor_SMD:R_0603_1608Metric, F.Cu at (18.2, 38.5)
- added R150: 150R, Resistor_SMD:R_0603_1608Metric, F.Cu at (18.2, 41.0)
- added R76: 150R, Resistor_SMD:R_0603_1608Metric, F.Cu at (325.6, 69.0)
- added R77: 10K, Resistor_SMD:R_0603_1608Metric, F.Cu at (306.5, 69.0)
- added R78: 150R, Resistor_SMD:R_0603_1608Metric, F.Cu at (306.5, 71.5)
- added R79: 10K, Resistor_SMD:R_0603_1608Metric, F.Cu at (325.6, 40.9)
- added R80: 150R, Resistor_SMD:R_0603_1608Metric, F.Cu at (325.6, 43.4)
- added R81: 10K, Resistor_SMD:R_0603_1608Metric, F.Cu at (319.2, 69.0)
- added R82: 150R, Resistor_SMD:R_0603_1608Metric, F.Cu at (319.2, 71.5)
- added R83: 10K, Resistor_SMD:R_0603_1608Metric, F.Cu at (312.9, 62.0)
- added R84: 150R, Resistor_SMD:R_0603_1608Metric, F.Cu at (312.9, 64.5)
- added R85: 10K, Resistor_SMD:R_0603_1608Metric, F.Cu at (306.5, 40.9)
- added R86: 150R, Resistor_SMD:R_0603_1608Metric, F.Cu at (306.5, 43.4)
- added R87: 10K, Resistor_SMD:R_0603_1608Metric, F.Cu at (306.5, 55.0)
- added R88: 150R, Resistor_SMD:R_0603_1608Metric, F.Cu at (306.5, 57.5)
- added R89: 10K, Resistor_SMD:R_0603_1608Metric, F.Cu at (306.5, 47.9)
- added R90: 150R, Resistor_SMD:R_0603_1608Metric, F.Cu at (306.5, 50.5)
- added R91: 10K, Resistor_SMD:R_0603_1608Metric, F.Cu at (319.2, 55.0)
- added R92: 150R, Resistor_SMD:R_0603_1608Metric, F.Cu at (319.2, 57.5)
- added R93: 10K, Resistor_SMD:R_0603_1608Metric, F.Cu at (283.7, 56.6)
- added R94: 150R, Resistor_SMD:R_0603_1608Metric, F.Cu at (283.7, 59.1)
- added R95: 10K, Resistor_SMD:R_0603_1608Metric, F.Cu at (325.6, 47.9)
- added R96: 150R, Resistor_SMD:R_0603_1608Metric, F.Cu at (325.6, 50.5)
- added R97: 10K, Resistor_SMD:R_0603_1608Metric, F.Cu at (300.2, 33.9)
- added R98: 150R, Resistor_SMD:R_0603_1608Metric, F.Cu at (300.2, 36.4)
- added R99: 10K, Resistor_SMD:R_0603_1608Metric, F.Cu at (312.9, 69.0)
- added U7: CP2102N-Axx-xQFN24, Package_DFN_QFN:QFN-24-1EP_4x4mm_P0.5mm_EP2.6x2.6mm, F.Cu at (285.1, 50.2)
- added U8: STM32F411RETx, Package_QFP:LQFP-64_10x10mm_P0.5mm, F.Cu at (288.8, 39.9)
- C1, C2, C3, C4: footprint Capacitor_THT:CP_Axial_L10.0mm_D4.5mm_P15.00mm_Horizontal -> Capacitor_SMD:C_0603_1608Metric
- C10, C11, C12, C13, C14, C15, C16, C17, C18, C19, C20, C21, C22, C23, C24, C25, C26, C27, C28, C29, C30, C31, C32, C33, C34, C35, C36, C37, C38, C39, C40, C41, C42, C43, C44, C45, C46, C47, C48, C49, C5, C50, C51, C52, C53, C54, C55, C56, C57, C58, C59, C6, C60, C61, C62, C63, C64, C65, C66, C67, C68, C69, C7, C70, C71, C8, C9: value C -> 1uF; footprint Capacitor_THT:CP_Axial_L10.0mm_D4.5mm_P15.00mm_Horizontal -> Capacitor_SMD:C_0603_1608Metric
- D1, D10, D11, D12, D13, D14, D15, D16, D17, D18, D19, D2, D20, D21, D22, D23, D24, D25, D26, D27, D28, D29, D3, D30, D31, D32, D33, D34, D35, D36, D37, D38, D39, D4, D40, D41, D42, D43, D44, D45, D46, D47, D48, D49, D5, D50, D51, D52, D53, D54, D55, D56, D57, D58, D59, D6, D60, D61, D62, D63, D64, D65, D66, D67, D7, D8, D9: value LED -> D_Schottky; footprint Diode_THT:D_DO-41_SOD81_P10.16mm_Horizontal -> Diode_SMD:D_SOD-123
- R1, R12, R13, R14, R15, R16, R17, R19, R21, R23, R25, R27, R29, R31, R33, R35, R37, R39, R4, R41, R43, R45, R47, R49, R51, R53, R55, R57, R59, R61, R63, R65, R67, R69, R7, R71, R73, R75, R8, R9: value R -> 10K
- R10: value R -> 4,7k
- R11: value R -> 4,7K
- R18, R20, R22, R24, R26, R28, R30, R32, R34, R36, R38, R40, R42, R44, R46, R48, R50, R52, R54, R56, R58, R60, R62, R64, R66, R68, R70, R72, R74: value R -> 150R
- R2: value R_Variable -> 10K; footprint Button_Switch_THT:Push_E-Switch_KS01Q01 -> Resistor_SMD:R_0603_1608Metric
- R3: value ~ -> 10K; footprint Resistor_THT:R_Axial_DIN0207_L6.3mm_D2.5mm_P7.62mm_Horizontal -> Resistor_SMD:R_0603_1608Metric
- R5: value R -> R_Variable; footprint Resistor_SMD:R_0603_1608Metric -> Button_Switch_THT:Push_E-Switch_KS01Q01
- R6: value R -> ~
- U3, U4, U5, U6: footprint Package_DIP:DIP-28_W7.62mm -> Package_SO:SOIC-28W_7.5x17.9mm_P1.27mm
Connections:
- D1 pad 1: /Button_RCD19/To_MCP_PIN -> Net-(D1-K)
- D1 pad 2: GND -> Net-(D1-A)
- D10 pad 1: /Button_RCD66/To_MCP_PIN -> Net-(D10-K)
- D10 pad 2: GND -> Net-(D10-A)
- D11 pad 1: /Button_RCD67/To_MCP_PIN -> Net-(D11-K)
- D11 pad 2: GND -> Net-(D11-A)
- D12 pad 1: /Button_RCD68/To_MCP_PIN -> Net-(D12-K)
- D12 pad 2: GND -> Net-(D12-A)
- D13 pad 1: /Button_RCD69/To_MCP_PIN -> Net-(D13-K)
- D13 pad 2: GND -> Net-(D13-A)
- D14 pad 1: /Button_RCD70/To_MCP_PIN -> Net-(D14-K)
- D14 pad 2: GND -> Net-(D14-A)
- D15 pad 1: /Button_RCD81/To_MCP_PIN -> Net-(D15-K)
- D15 pad 2: GND -> Net-(D15-A)
- D16 pad 1: /Button_RCD79/To_MCP_PIN -> Net-(D16-K)
- D16 pad 2: GND -> Net-(D16-A)
- D17 pad 1: /Button_RCD16/To_MCP_PIN -> Net-(D17-K)
- D17 pad 2: GND -> Net-(D17-A)
- D18 pad 1: /Button_RCD17/To_MCP_PIN -> Net-(D18-K)
- D18 pad 2: GND -> Net-(D18-A)
- D19 pad 1: /Button_RCD18/To_MCP_PIN -> Net-(D19-K)
- D19 pad 2: GND -> Net-(D19-A)
- D2 pad 1: /Button_RCD71/To_MCP_PIN -> Net-(D2-K)
- D2 pad 2: GND -> Net-(D2-A)
- D20 pad 1: /Button_RCD80/To_MCP_PIN -> Net-(D20-K)
- D20 pad 2: GND -> Net-(D20-A)
- D21 pad 1: /Button_RCD20/To_MCP_PIN -> Net-(D21-K)
- D21 pad 2: GND -> Net-(D21-A)
- D22 pad 1: /Button_RCD21/To_MCP_PIN -> Net-(D22-K)
- D22 pad 2: GND -> Net-(D22-A)
- D23 pad 1: /Button_RCD22/To_MCP_PIN -> Net-(D23-K)
- D23 pad 2: GND -> Net-(D23-A)
- D24 pad 1: /Button_RCD23/To_MCP_PIN -> Net-(D24-K)
- D24 pad 2: GND -> Net-(D24-A)
- D25 pad 1: /Button_RCD24/To_MCP_PIN -> Net-(D25-K)
- D25 pad 2: GND -> Net-(D25-A)
- D26 pad 1: /Button_RCD25/To_MCP_PIN -> Net-(D26-K)
- D26 pad 2: GND -> Net-(D26-A)
- D27 pad 1: /Button_RCD26/To_MCP_PIN -> Net-(D27-K)
- D27 pad 2: GND -> Net-(D27-A)
- D28 pad 1: /Button_RCD27/To_MCP_PIN -> Net-(D28-K)
- D28 pad 2: GND -> Net-(D28-A)
- D29 pad 1: /Button_RCD28/To_MCP_PIN -> Net-(D29-K)
- D29 pad 2: GND -> Net-(D29-A)
- D3 pad 1: /Button_RCD72/To_MCP_PIN -> Net-(D3-K)
- D3 pad 2: GND -> Net-(D3-A)
- D30 pad 1: /Button_RCD29/To_MCP_PIN -> Net-(D30-K)
- D30 pad 2: GND -> Net-(D30-A)
- D31 pad 1: /Button_RCD30/To_MCP_PIN -> Net-(D31-K)
- D31 pad 2: GND -> Net-(D31-A)
- D32 pad 1: /Button_RCD31/To_MCP_PIN -> Net-(D32-K)
- D32 pad 2: GND -> Net-(D32-A)
- D33 pad 1: /Button_RCD32/To_MCP_PIN -> Net-(D33-K)
- D33 pad 2: GND -> Net-(D33-A)
- D34 pad 1: /Button_RCD33/To_MCP_PIN -> Net-(D34-K)
- D34 pad 2: GND -> Net-(D34-A)
- D35 pad 1: /Button_RCD34/To_MCP_PIN -> Net-(D35-K)
- D35 pad 2: GND -> Net-(D35-A)
- D36 pad 1: /Button_RCD35/To_MCP_PIN -> Net-(D36-K)
- D36 pad 2: GND -> Net-(D36-A)
- D37 pad 1: /Button_RCD36/To_MCP_PIN -> Net-(D37-K)
- D37 pad 2: GND -> Net-(D37-A)
- D38 pad 1: /Button_RCD37/To_MCP_PIN -> Net-(D38-K)
- D38 pad 2: GND -> Net-(D38-A)
- D39 pad 1: /Button_RCD38/To_MCP_PIN -> Net-(D39-K)
- D39 pad 2: GND -> Net-(D39-A)
- D4 pad 1: /Button_RCD73/To_MCP_PIN -> Net-(D4-K)
- D4 pad 2: GND -> Net-(D4-A)
- D40 pad 1: /Button_RCD39/To_MCP_PIN -> Net-(D40-K)
- D40 pad 2: GND -> Net-(D40-A)
- D41 pad 1: /Button_RCD40/To_MCP_PIN -> Net-(D41-K)
- D41 pad 2: GND -> Net-(D41-A)
- D42 pad 1: /Button_RCD41/To_MCP_PIN -> Net-(D42-K)
- D42 pad 2: GND -> Net-(D42-A)
- D43 pad 1: /Button_RCD42/To_MCP_PIN -> Net-(D43-K)
- D43 pad 2: GND -> Net-(D43-A)
- D44 pad 1: /Button_RCD43/To_MCP_PIN -> Net-(D44-K)
- D44 pad 2: GND -> Net-(D44-A)
- D45 pad 1: /Button_RCD44/To_MCP_PIN -> Net-(D45-K)
- D45 pad 2: GND -> Net-(D45-A)
- D46 pad 1: /Button_RCD45/To_MCP_PIN -> Net-(D46-K)
- D46 pad 2: GND -> Net-(D46-A)
- D47 pad 1: /Button_RCD83/To_MCP_PIN -> Net-(D47-K)
- D47 pad 2: GND -> Net-(D47-A)
- D48 pad 1: /Button_RCD47/To_MCP_PIN -> Net-(D48-K)
- D48 pad 2: GND -> Net-(D48-A)
- D49 pad 1: /Button_RCD46/To_MCP_PIN -> Net-(D49-K)
- D49 pad 2: GND -> Net-(D49-A)
- D5 pad 1: /Button_RCD74/To_MCP_PIN -> Net-(D5-K)
- D5 pad 2: GND -> Net-(D5-A)
- D50 pad 1: /Button_RCD48/To_MCP_PIN -> Net-(D50-K)
- D50 pad 2: GND -> Net-(D50-A)
- D51 pad 1: /Button_RCD49/To_MCP_PIN -> Net-(D51-K)
- D51 pad 2: GND -> Net-(D51-A)
- D52 pad 1: /Button_RCD50/To_MCP_PIN -> Net-(D52-K)
- D52 pad 2: GND -> Net-(D52-A)
- D53 pad 1: /Button_RCD51/To_MCP_PIN -> Net-(D53-K)
- D53 pad 2: GND -> Net-(D53-A)
- D54 pad 1: /Button_RCD52/To_MCP_PIN -> Net-(D54-K)
- D54 pad 2: GND -> Net-(D54-A)
- D55 pad 1: /Button_RCD53/To_MCP_PIN -> Net-(D55-K)
- D55 pad 2: GND -> Net-(D55-A)
- D56 pad 1: /Button_RCD55/To_MCP_PIN -> Net-(D56-K)
- D56 pad 2: GND -> Net-(D56-A)
- D57 pad 1: /Button_RCD56/To_MCP_PIN -> Net-(D57-K)
- D57 pad 2: GND -> Net-(D57-A)
- D58 pad 1: /Button_RCD57/To_MCP_PIN -> Net-(D58-K)
- D58 pad 2: GND -> Net-(D58-A)
- D59 pad 1: /Button_RCD58/To_MCP_PIN -> Net-(D59-K)
- D59 pad 2: GND -> Net-(D59-A)
- D6 pad 1: /Button_RCD75/To_MCP_PIN -> Net-(D6-K)
- D6 pad 2: GND -> Net-(D6-A)
- D60 pad 1: /Button_RCD59/To_MCP_PIN -> Net-(D60-K)
- D60 pad 2: GND -> Net-(D60-A)
- D61 pad 1: /Button_RCD60/To_MCP_PIN -> Net-(D61-K)
- D61 pad 2: GND -> Net-(D61-A)
- D62 pad 1: /Button_RCD61/To_MCP_PIN -> Net-(D62-K)
- D62 pad 2: GND -> Net-(D62-A)
- D63 pad 1: /Button_RCD85/To_MCP_PIN -> Net-(D63-K)
- D63 pad 2: GND -> Net-(D63-A)
- D64 pad 1: /Button_RCD63/To_MCP_PIN -> Net-(D64-K)
- D64 pad 2: GND -> Net-(D64-A)
- D65 pad 1: /Button_RCD82/To_MCP_PIN -> Net-(D65-K)
- D65 pad 2: GND -> Net-(D65-A)
- D66 pad 1: /Button_RCD84/To_MCP_PIN -> Net-(D66-K)
- D66 pad 2: GND -> Net-(D66-A)
- D67 pad 1: /Button_RCD86/To_MCP_PIN -> Net-(D67-K)
- D67 pad 2: GND -> Net-(D67-A)
- D7 pad 1: /Button_RCD76/To_MCP_PIN -> Net-(D7-K)
- D7 pad 2: GND -> Net-(D7-A)
- D8 pad 1: /Button_RCD64/To_MCP_PIN -> Net-(D8-K)
- D8 pad 2: GND -> Net-(D8-A)
- D9 pad 1: /Button_RCD65/To_MCP_PIN -> Net-(D9-K)
- D9 pad 2: GND -> Net-(D9-A)
- R1 pad 2: Net-(U3-~{RESET}) -> Net-(U2-PA10)
- R10 pad 1: /Button_RCD71/To_MCP_PIN -> +3.3V
- R10 pad 2: GND -> /SCL
- R11 pad 1: /Button_RCD72/To_MCP_PIN -> +3.3V
- R11 pad 2: GND -> /SDA
- R12 pad 1: /Button_RCD73/To_MCP_PIN -> +3.3V
- R12 pad 2: GND -> Net-(U5-INTB)
- R13 pad 1: /Button_RCD74/To_MCP_PIN -> +3.3V
- R13 pad 2: GND -> Net-(U5-~{RESET})
- R14 pad 1: /Button_RCD75/To_MCP_PIN -> +3.3V
- R14 pad 2: GND -> Net-(U6-INTB)
- R15 pad 1: /Button_RCD76/To_MCP_PIN -> +3.3V
- R15 pad 2: GND -> Net-(U6-~{RESET})
- R16 pad 1: /Button_RCD64/To_MCP_PIN -> +3.3V
- R16 pad 2: GND -> Net-(U2-PA10)
- R17 pad 1: /Button_RCD65/To_MCP_PIN -> +3.3V
- R17 pad 2: GND -> /Button_RCD19/To_MCP_PIN
- R18 pad 1: /Button_RCD66/To_MCP_PIN -> /Button_RCD19/To_MCP_PIN
- R18 pad 2: GND -> Net-(D1-A)
- R19 pad 1: /Button_RCD67/To_MCP_PIN -> +3.3V
- R19 pad 2: GND -> /Button_RCD71/To_MCP_PIN
- R2 pad 2: Net-(U2-PA1) -> Net-(U3-INTB)
- R20 pad 1: /Button_RCD68/To_MCP_PIN -> /Button_RCD71/To_MCP_PIN
- R20 pad 2: GND -> Net-(D2-A)
- R21 pad 1: /Button_RCD69/To_MCP_PIN -> +3.3V
- R21 pad 2: GND -> /Button_RCD72/To_MCP_PIN
- R22 pad 1: /Button_RCD70/To_MCP_PIN -> /Button_RCD72/To_MCP_PIN
- R22 pad 2: GND -> Net-(D3-A)
- R23 pad 1: /Button_RCD81/To_MCP_PIN -> +3.3V
- R23 pad 2: GND -> /Button_RCD73/To_MCP_PIN
- R24 pad 1: /Button_RCD79/To_MCP_PIN -> /Button_RCD73/To_MCP_PIN
- R24 pad 2: GND -> Net-(D4-A)
- R25 pad 1: /Button_RCD16/To_MCP_PIN -> +3.3V
- R25 pad 2: GND -> /Button_RCD74/To_MCP_PIN
- R26 pad 1: /Button_RCD17/To_MCP_PIN -> /Button_RCD74/To_MCP_PIN
- R26 pad 2: GND -> Net-(D5-A)
- R27 pad 1: /Button_RCD18/To_MCP_PIN -> +3.3V
- R27 pad 2: GND -> /Button_RCD75/To_MCP_PIN
- R28 pad 1: /Button_RCD80/To_MCP_PIN -> /Button_RCD75/To_MCP_PIN
- R28 pad 2: GND -> Net-(D6-A)
- R29 pad 1: /Button_RCD20/To_MCP_PIN -> +3.3V
- R29 pad 2: GND -> /Button_RCD76/To_MCP_PIN
- R3 pad 1: Net-(U2-PA1) -> +3.3V
- R3 pad 2: GND -> Net-(U3-~{RESET})
- R30 pad 1: /Button_RCD21/To_MCP_PIN -> /Button_RCD76/To_MCP_PIN
- R30 pad 2: GND -> Net-(D7-A)
- R31 pad 1: /Button_RCD22/To_MCP_PIN -> +3.3V
- R31 pad 2: GND -> /Button_RCD64/To_MCP_PIN
- R32 pad 1: /Button_RCD23/To_MCP_PIN -> /Button_RCD64/To_MCP_PIN
- R32 pad 2: GND -> Net-(D8-A)
- R33 pad 1: /Button_RCD24/To_MCP_PIN -> +3.3V
- R33 pad 2: GND -> /Button_RCD65/To_MCP_PIN
- R34 pad 1: /Button_RCD25/To_MCP_PIN -> /Button_RCD65/To_MCP_PIN
- R34 pad 2: GND -> Net-(D9-A)
- R35 pad 1: /Button_RCD26/To_MCP_PIN -> +3.3V
- R35 pad 2: GND -> /Button_RCD66/To_MCP_PIN
- R36 pad 1: /Button_RCD27/To_MCP_PIN -> /Button_RCD66/To_MCP_PIN
- R36 pad 2: GND -> Net-(D10-A)
- R37 pad 1: /Button_RCD28/To_MCP_PIN -> +3.3V
- R37 pad 2: GND -> /Button_RCD67/To_MCP_PIN
- R38 pad 1: /Button_RCD29/To_MCP_PIN -> /Button_RCD67/To_MCP_PIN
- R38 pad 2: GND -> Net-(D11-A)
- R39 pad 1: /Button_RCD30/To_MCP_PIN -> +3.3V
- R39 pad 2: GND -> /Button_RCD68/To_MCP_PIN
- R4 pad 2: Net-(U4-~{RESET}) -> Net-(U2-PA10)
- R40 pad 1: /Button_RCD31/To_MCP_PIN -> /Button_RCD68/To_MCP_PIN
- R40 pad 2: GND -> Net-(D12-A)
- R41 pad 1: /Button_RCD32/To_MCP_PIN -> +3.3V
- R41 pad 2: GND -> /Button_RCD69/To_MCP_PIN
- R42 pad 1: /Button_RCD33/To_MCP_PIN -> /Button_RCD69/To_MCP_PIN
- R42 pad 2: GND -> Net-(D13-A)
- R43 pad 1: /Button_RCD34/To_MCP_PIN -> +3.3V
- R43 pad 2: GND -> /Button_RCD70/To_MCP_PIN
- R44 pad 1: /Button_RCD35/To_MCP_PIN -> /Button_RCD70/To_MCP_PIN
- R44 pad 2: GND -> Net-(D14-A)
- R45 pad 1: /Button_RCD36/To_MCP_PIN -> +3.3V
- R45 pad 2: GND -> /Button_RCD81/To_MCP_PIN
- R46 pad 1: /Button_RCD37/To_MCP_PIN -> /Button_RCD81/To_MCP_PIN
- R46 pad 2: GND -> Net-(D15-A)
- R47 pad 1: /Button_RCD38/To_MCP_PIN -> +3.3V
- R47 pad 2: GND -> /Button_RCD79/To_MCP_PIN
- R48 pad 1: /Button_RCD39/To_MCP_PIN -> /Button_RCD79/To_MCP_PIN
- R48 pad 2: GND -> Net-(D16-A)
- R49 pad 1: /Button_RCD40/To_MCP_PIN -> +3.3V
- R49 pad 2: GND -> /Button_RCD16/To_MCP_PIN
- R5 pad 2: Net-(U2-PB8) -> Net-(U2-PA1)
- R50 pad 1: /Button_RCD41/To_MCP_PIN -> /Button_RCD16/To_MCP_PIN
- R50 pad 2: GND -> Net-(D17-A)
- R51 pad 1: /Button_RCD42/To_MCP_PIN -> +3.3V
- R51 pad 2: GND -> /Button_RCD17/To_MCP_PIN
- R52 pad 1: /Button_RCD43/To_MCP_PIN -> /Button_RCD17/To_MCP_PIN
- R52 pad 2: GND -> Net-(D18-A)
- R53 pad 1: /Button_RCD44/To_MCP_PIN -> +3.3V
- R53 pad 2: GND -> /Button_RCD18/To_MCP_PIN
- R54 pad 1: /Button_RCD45/To_MCP_PIN -> /Button_RCD18/To_MCP_PIN
- R54 pad 2: GND -> Net-(D19-A)
- R55 pad 1: /Button_RCD83/To_MCP_PIN -> +3.3V
- R55 pad 2: GND -> /Button_RCD80/To_MCP_PIN
- R56 pad 1: /Button_RCD47/To_MCP_PIN -> /Button_RCD80/To_MCP_PIN
- R56 pad 2: GND -> Net-(D20-A)
- R57 pad 1: /Button_RCD46/To_MCP_PIN -> +3.3V
- R57 pad 2: GND -> /Button_RCD20/To_MCP_PIN
- R58 pad 1: /Button_RCD48/To_MCP_PIN -> /Button_RCD20/To_MCP_PIN
- R58 pad 2: GND -> Net-(D21-A)
- R59 pad 1: /Button_RCD49/To_MCP_PIN -> +3.3V
- R59 pad 2: GND -> /Button_RCD21/To_MCP_PIN
- R6 pad 1: +3.3V -> Net-(U2-PA1)
- R6 pad 2: Net-(U2-PB9) -> GND
- R60 pad 1: /Button_RCD50/To_MCP_PIN -> /Button_RCD21/To_MCP_PIN
- R60 pad 2: GND -> Net-(D22-A)
- R61 pad 1: /Button_RCD51/To_MCP_PIN -> +3.3V
- R61 pad 2: GND -> /Button_RCD22/To_MCP_PIN
- R62 pad 1: /Button_RCD52/To_MCP_PIN -> /Button_RCD22/To_MCP_PIN
- R62 pad 2: GND -> Net-(D23-A)
- R63 pad 1: /Button_RCD53/To_MCP_PIN -> +3.3V
- R63 pad 2: GND -> /Button_RCD23/To_MCP_PIN
- R64 pad 1: /Button_RCD55/To_MCP_PIN -> /Button_RCD23/To_MCP_PIN
- R64 pad 2: GND -> Net-(D24-A)
- R65 pad 1: /Button_RCD56/To_MCP_PIN -> +3.3V
- R65 pad 2: GND -> /Button_RCD24/To_MCP_PIN
- R66 pad 1: /Button_RCD57/To_MCP_PIN -> /Button_RCD24/To_MCP_PIN
- R66 pad 2: GND -> Net-(D25-A)
- R67 pad 1: /Button_RCD58/To_MCP_PIN -> +3.3V
- R67 pad 2: GND -> /Button_RCD25/To_MCP_PIN
- R68 pad 1: /Button_RCD59/To_MCP_PIN -> /Button_RCD25/To_MCP_PIN
- R68 pad 2: GND -> Net-(D26-A)
- R69 pad 1: /Button_RCD60/To_MCP_PIN -> +3.3V
- R69 pad 2: GND -> /Button_RCD26/To_MCP_PIN
- R7 pad 2: Net-(U5-~{RESET}) -> Net-(U4-INTB)
- R70 pad 1: /Button_RCD61/To_MCP_PIN -> /Button_RCD26/To_MCP_PIN
- R70 pad 2: GND -> Net-(D27-A)
- R71 pad 1: /Button_RCD85/To_MCP_PIN -> +3.3V
- R71 pad 2: GND -> /Button_RCD27/To_MCP_PIN
- R72 pad 1: /Button_RCD63/To_MCP_PIN -> /Button_RCD27/To_MCP_PIN
- R72 pad 2: GND -> Net-(D28-A)
- R73 pad 1: /Button_RCD82/To_MCP_PIN -> +3.3V
- R73 pad 2: GND -> /Button_RCD28/To_MCP_PIN
- R74 pad 1: /Button_RCD84/To_MCP_PIN -> /Button_RCD28/To_MCP_PIN
- R74 pad 2: GND -> Net-(D29-A)
- R75 pad 1: /Button_RCD86/To_MCP_PIN -> +3.3V
- R75 pad 2: GND -> /Button_RCD29/To_MCP_PIN
- R8 pad 2: Net-(U6-~{RESET}) -> Net-(U4-~{RESET})
- R9 pad 1: /Button_RCD19/To_MCP_PIN -> +3.3V
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