File: kicadProjects/0511/0511/0511.kicad_pcb (KiCad board)
At the start: 2 copper layers, 304.2 x 286.5 mm, 379 parts, among them J1 USB4120-03-C_REVA6, U1 UDA1334A_Breakout, U2 STM32F411RETx, U3 BD33HC5WEFJ-E2, Y1 32.768KHz, Y2 8MHz

Commit message: poursuite placement
Parts:
- moved C73 53.8 mm to (211.8, 97.6), turned to -90 degrees
- moved U3 53.4 mm to (214.6, 93.4)
- moved C74 51.5 mm to (203.8, 99.8)
- moved C75 51.5 mm to (197.1, 98.7)
- moved C76 51.5 mm to (199.7, 89.0)
- moved R131 51.5 mm to (201.2, 99.8)
- moved R133 51.5 mm to (206.7, 100.7)
- moved C77 51.5 mm to (206.7, 98.9)
- moved CR1 51.5 mm to (197.1, 101.3)
- moved J1 51.5 mm to (201.8, 93.8)
- moved R132 51.5 mm to (199.7, 87.3)
- moved JST_PH_FEMALE_FSR1 45.6 mm to (125.2, 41.7)
- moved C5 45.6 mm to (100.0, 49.8)
- moved D1 45.6 mm to (105.4, 53.4)
- moved JST_PH_FEMAILE_PUSH_BUTTON1 45.6 mm to (103.4, 41.5)
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Routing:
- net /Stm32f411retx/PA11: track 65.1 -> 25.3 mm
- net /Stm32f411retx/PA12: track 70.2 -> 30.8 mm
- net VBUS_A: track 3.12 -> 12.4 mm, vias 0 -> 2
- net +3.3V: track 280.4 -> 282.6 mm
- net GND: track 27.9 -> 30.0 mm

Commit message: poursuite
Parts:
- moved A6_23 70.8 mm to (193.5, 52.1), turned to 180 degrees
- moved A6_23_R1 59.7 mm to (202.2, 65.0), turned to 90 degrees
- moved A6_23_D1 32.8 mm to (212.7, 49.0), turned to -90 degrees

Commit message: ajout rail alim
Parts:
- moved C76 80.3 mm to (140.8, 34.3), turned to 180 degrees
- moved C75 80.3 mm to (142.3, 39.9)
- moved C77 80.3 mm to (151.9, 40.1)
- moved CR1 80.3 mm to (142.3, 42.5)
- moved J1 80.3 mm to (147.1, 35.0)
- moved R133 80.3 mm to (151.9, 41.9)
- moved C74 79.7 mm to (149.0, 42.0)
- moved R131 79.2 mm to (147.2, 42.0)
- moved C73 78.6 mm to (159.0, 39.4)
- moved C68 78.6 mm to (166.4, 35.8)
- moved U3 78.6 mm to (161.8, 35.2)
- moved R132 78.0 mm to (140.9, 36.0), turned to 180 degrees
- moved D58 76.1 mm to (145.8, 39.4), turned to -90 degrees
- moved D59 73.5 mm to (148.2, 39.4), turned to -90 degrees
- moved U2 37.4 mm to (147.2, 73.4)
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Routing:
- net +3.3V: track 282.6 -> 552.1 mm, vias 0 -> 7
- net /SDA: track 283.2 -> 349.2 mm, vias 5 -> 6
- net /FSR: track 59.1 -> 9.69 mm
- net /Stm32f411retx/PA11: track 25.3 -> 48.8 mm
- net /Stm32f411retx/PA12: track 30.8 -> 46.4 mm
- net Net-(C76-Pad1): track 4.62 -> 19.6 mm, vias 0 -> 2
- net Net-(J1-CC1): track 0.00 -> 10.3 mm
- net VBUS_A: track 12.4 -> 18.5 mm, vias 2 -> 4
- net /Stm32f411retx/SWDIO: track 17.7 -> 19.2 mm

Commit message: poursuite alim
Parts:
- moved D58 7.82 mm to (152.4, 35.2)
- moved A6_23_D1 4.82 mm to (208.0, 50.2)
- moved A6_23_R1 4.64 mm to (208.0, 54.8)
Routing:
- net +3.3V: track 552.1 -> 713.3 mm, vias 7 -> 19
- net /MOSI: track 0.00 -> 131.3 mm, vias 0 -> 2
- net /BCLCK: track 0.00 -> 129.9 mm, vias 0 -> 2
- net /WSEL: track 0.00 -> 126.2 mm, vias 0 -> 2
- net /Button_RCD46/To_MCP_PIN: track 14.4 -> 132.1 mm, vias 0 -> 2
- net /SDA: track 349.2 -> 317.0 mm
- net VBUS_A: track 18.5 -> 31.5 mm, vias 4 -> 6
- net Net-(A6_23_D1-K): track 0.00 -> 8.60 mm
- net /Stm32f411retx/PA11: track 48.8 -> 52.9 mm, vias 2 -> 3
- net Net-(A6_23_D1-A): track 0.00 -> 2.10 mm

Commit message: poursuite placement
Parts:
- moved RESET_PULLUP_22 19.5 mm to (173.6, 259.6), turned to -90 degrees
Routing:
- net +3.3V: track 713.3 -> 883.1 mm, vias 19 -> 32
- net /FSR: track 9.69 -> 55.7 mm
- net Net-(MCP23017_ADD22-INTB): track 0.00 -> 5.80 mm
- net /INT3: track 0.00 -> 4.79 mm
- net Net-(MCP23017_ADD22-~{RESET}): track 0.00 -> 4.73 mm, vias 0 -> 2
- net GND: track 30.0 -> 31.0 mm
- net /Stm32f411retx/NRST: track 7.28 -> 8.29 mm
- net /SDA: track 317.0 -> 316.2 mm, vias 6 -> 5

Commit message: poursuite cablage
Parts:
- added REF**: MountingHole_3.2mm_M3, MountingHole:MountingHole_3.2mm_M3, F.Cu at (19.6, 39.4)
- added REF**: MountingHole_3.2mm_M3, MountingHole:MountingHole_3.2mm_M3, F.Cu at (309.0, 39.2)
- added REF**: MountingHole_3.2mm_M3, MountingHole:MountingHole_3.2mm_M3, F.Cu at (24.8, 309.8)
- added REF**: MountingHole_3.2mm_M3, MountingHole:MountingHole_3.2mm_M3, F.Cu at (306.8, 307.2)
- moved A6_23 27.5 mm to (220.9, 49.9)
- moved U1 24.5 mm to (56.4, 46.3)
- moved A6_23_R1 18.7 mm to (221.4, 67.8)
- moved A6_23_D1 18.7 mm to (221.4, 63.2)
Routing:
- net +3.3V: track 883.1 -> 859.5 mm
- net Net-(A6_23_D1-K): track 8.60 -> 16.6 mm
- net /Button_RCD46/To_MCP_PIN: track 132.1 -> 124.7 mm
- net /WSEL: track 126.2 -> 130.0 mm
- net /MOSI: track 131.3 -> 129.8 mm
- net /BCLCK: track 129.9 -> 131.1 mm
- net /SDA: track 316.2 -> 315.3 mm
