File: kicadProjects/0511/0511/0511.kicad_sch (KiCad schematic)
At the start: 27 parts, among them U1 UDA1334A_Breakout, U2 YAAJ_BlackPill, U3 MCP23017, U4 MCP23017, U5 MCP23017, U6 MCP23017, U7 CP2102N-Axx-xQFN24

Commit message: poursuite
Connections:
- net at U2.27 (PA4): no longer U1.4 (WSEL)
- net at U2.28 (PA5): no longer U1.5 (BCLK)
- net at U2.30 (PA7): no longer U1.6 (DIN)
- new net BCLCK: U1.5 (BCLK)
- new net MOSI: U1.6 (DIN)
- new net WSEL: U1.4 (WSEL)
Other:
- sheet Stm32f411retx ports: added BCLCK, WSEL; removed none
Changed lines of the file:
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@@
 	(wire
 		(pts
-			(xy 36.83 11.43) (xy 36.83 44.45)
+			(xy 264.16 63.5) (xy 264.16 69.85)
 		)
 		(stroke
@@
 	(wire
 		(pts
-			(xy 264.16 63.5) (xy 264.16 69.85)
+			(xy 246.38 58.42) (xy 246.38 60.96)
 		)
 		(stroke
@@
 	(wire
 		(pts
-			(xy 246.38 58.42) (xy 246.38 60.96)
+			(xy 248.92 209.55) (xy 248.92 214.63)
 		)
 		(stroke
@@
 	(wire
 		(pts
-			(xy 177.8 48.26) (xy 177.8 11.43)
-		)
-		(stroke
-			(width 0)
-			(type default)
-		)
-	)
-	(wire
-		(pts
 			(xy 218.44 138.43) (xy 238.76 138.43)
 		)
@@
 	(wire
 		(pts
-			(xy 43.18 16.51) (xy 182.88 16.51)
-		)
-		(stroke
-			(width 0)
-			(type default)
-		)
-	)
-	(wire
-		(pts
 			(xy 339.09 115.57) (xy 342.9 115.57)
 		)
@@
 	(wire
 		(pts
-			(xy 165.1 50.8) (xy 182.88 50.8)
+			(xy 85.09 134.62) (xy 85.09 154.94)
 		)
 		(stroke
@@
 	(wire
 		(pts
-			(xy 85.09 134.62) (xy 85.09 154.94)
+			(xy 281.94 92.71) (xy 281.94 87.63)
 		)
 		(stroke
@@
 	(wire
 		(pts
-			(xy 281.94 92.71) (xy 281.94 87.63)
+			(xy 39.37 161.29) (xy 39.37 162.56)
 		)
 		(stroke
@@
 	(wire
 		(pts
-			(xy 39.37 161.29) (xy 39.37 162.56)
+			(xy 227.33 223.52) (xy 234.95 223.52)
 		)
 		(stroke
@@
 	(wire
 		(pts
-			(xy 167.64 156.21) (xy 172.72 156.21)
+			(xy 44.45 41.91) (xy 62.23 41.91)
 		)
 		(stroke
@@
 	(wire
 		(pts
-			(xy 158.75 171.45) (xy 158.75 160.02)
+			(xy 167.64 156.21) (xy 172.72 156.21)
 		)
 		(stroke
@@
 	(wire
 		(pts
-			(xy 36.83 44.45) (xy 62.23 44.45)
+			(xy 158.75 171.45) (xy 158.75 160.02)
 		)
 		(stroke
@@
 	(wire
 		(pts
-			(xy 255.27 105.41) (xy 254 105.41)
+			(xy 44.45 44.45) (xy 62.23 44.45)
 		)
 		(stroke
@@
 	(wire
 		(pts
-			(xy 87.63 147.32) (xy 92.71 147.32)
+			(xy 255.27 105.41) (xy 254 105.41)
 		)
 		(stroke
@@
 	(wire
 		(pts
-			(xy 82.55 151.13) (xy 82.55 134.62)
+			(xy 87.63 147.32) (xy 92.71 147.32)
 		)
 		(stroke
@@
 	(wire
 		(pts
-			(xy 34.29 116.84) (xy 41.91 116.84)
+			(xy 82.55 151.13) (xy 82.55 134.62)
 		)
 		(stroke
@@
 	(wire
 		(pts
-			(xy 62.23 134.62) (xy 62.23 161.29)
+			(xy 34.29 116.84) (xy 41.91 116.84)
 		)
 		(stroke
@@
 	(wire
 		(pts
-			(xy 57.15 134.62) (xy 57.15 171.45)
+			(xy 62.23 134.62) (xy 62.23 161.29)
 		)
 		(stroke
@@
 	(wire
 		(pts
-			(xy 85.09 71.12) (xy 85.09 76.2)
+			(xy 57.15 134.62) (xy 57.15 171.45)
 		)
 		(stroke
@@
 	(wire
 		(pts
-			(xy 165.1 48.26) (xy 177.8 48.26)
+			(xy 85.09 71.12) (xy 85.09 76.2)
 		)
 		(stroke
@@
 	(wire
 		(pts
-			(xy 119.38 39.37) (xy 119.38 19.05)
-		)
-		(stroke
-			(width 0)
-			(type default)
-		)
-	)
-	(wire
-		(pts
 			(xy 364.49 95.25) (xy 360.68 95.25)
 		)
@@
 	(wire
 		(pts
-			(xy 177.8 11.43) (xy 36.83 11.43)
-		)
-		(stroke
-			(width 0)
-			(type default)
-		)
-	)
-	(wire
-		(pts
 			(xy 165.1 58.42) (xy 187.96 58.42)
 		)
@@
 	(wire
 		(pts
-			(xy 182.88 16.51) (xy 182.88 50.8)
-		)
-		(stroke
-			(width 0)
-			(type default)
-		)
-	)
-	(wire
-		(pts
 			(xy 191.77 53.34) (xy 191.77 57.15)
 		)
@@
 	(wire
 		(pts
-			(xy 43.18 41.91) (xy 62.23 41.91)
-		)
-		(stroke
-			(width 0)
-			(type default)
-		)
-	)
-	(wire
-		(pts
 			(xy 90.17 71.12) (xy 90.17 76.2)
 		)
@@
 	(wire
 		(pts
-			(xy 167.64 19.05) (xy 167.64 43.18)
-		)
-		(stroke
-			(width 0)
-			(type default)
-		)
-	)
-	(wire
-		(pts
 			(xy 62.23 39.37) (xy 62.23 38.1)
 		)
@@
 	(wire
 		(pts
-			(xy 77.47 39.37) (xy 119.38 39.37)
-		)
-		(stroke
-			(width 0)
-			(type default)
-		)
-	)
-	(wire
-		(pts
 			(xy 234.95 234.95) (xy 226.06 234.95)
 		)
@@
 	(wire
 		(pts
-			(xy 77.47 39.37) (xy 77.47 36.83)
+			(xy 77.47 36.83) (xy 77.47 40.64)
 		)
 		(stroke
@@
 	(wire
 		(pts
-			(xy 119.38 19.05) (xy 167.64 19.05)
-		)
-		(stroke
-			(width 0)
-			(type default)
-		)
-	)
-	(wire
-		(pts
 			(xy 217.17 77.47) (xy 217.17 80.01)
 		)
@@
 	(wire
 		(pts
+			(xy 252.73 223.52) (xy 257.81 223.52)
+		)
+		(stroke
+			(width 0)
+			(type default)
+		)
+	)
+	(wire
+		(pts
 			(xy 132.08 143.51) (xy 132.08 196.85)
 		)
@@
 	(wire
 		(pts
+			(xy 83.82 40.64) (xy 77.47 40.64)
+		)
+		(stroke
+			(width 0)
+			(type default)
+		)
+	)
+	(wire
+		(pts
 			(xy 134.62 143.51) (xy 134.62 185.42)
 		)
@@
 	(wire
 		(pts
-			(xy 43.18 16.51) (xy 43.18 41.91)
-		)
-		(stroke
-			(width 0)
-			(type default)
-		)
-	)
-	(wire
-		(pts
 			(xy 133.35 43.18) (xy 124.46 43.18)
 		)
@@
 		)
 	)
+	(label "BCLCK"
+		(at 257.81 223.52 0)
+		(effects
+			(font
+				(size 1.27 1.27)
+			)
+			(justify left bottom)
+		)
+	)
+	(label "WSEL"
+		(at 248.92 209.55 0)
+		(effects
+			(font
+				(size 1.27 1.27)
+			)
+			(justify left bottom)
+		)
+	)
 	(label "SDA"
 		(at 372.11 36.83 90)
@@
 		)
 	)
+	(label "BCLCK"
+		(at 44.45 44.45 0)
+		(effects
+			(font
+				(size 1.27 1.27)
+			)
+			(justify left bottom)
+		)
+	)
 	(label "SCL"
 		(at 85.09 95.25 0)
@@
 		)
 	)
+	(label "MOSI"
+		(at 83.82 40.64 0)
+		(effects
+			(font
+				(size 1.27 1.27)
+			)
+			(justify left bottom)
+		)
+	)
 	(label "SDA"
 		(at 90.17 95.25 0)
@@
 		)
 	)
+	(label "MOSI"
+		(at 227.33 223.52 0)
+		(effects
+			(font
+				(size 1.27 1.27)
+			)
+			(justify left bottom)
+		)
+	)
 	(label "INT4"
 		(at 332.74 22.86 0)
@@
 		)
 	)
+	(label "WSEL"
+		(at 44.45 41.91 0)
+		(effects
+			(font
+				(size 1.27 1.27)
+			)
+			(justify left bottom)
+		)
+	)
 	(label "INT3"
 		(at 247.65 43.18 0)
@@
 			)
 		)
+		(pin "WSEL" bidirectional
+			(at 248.92 214.63 90)
+			(effects
+				(font
+					(size 1.27 1.27)
+				)
+				(justify right)
+			)
+		)
+		(pin "BCLCK" bidirectional
+			(at 252.73 223.52 0)
+			(effects
+				(font
+					(size 1.27 1.27)
+				)
+				(justify right)
+			)
+		)

Commit message: assignation empreintes
Parts:
- removed U2: YAAJ_BlackPill, Footprints:YAAJ_BlackPill_SWD_1, symbol Stm32F411BlackPill:YAAJ_BlackPill
- renumbered C3 to C2, C2 to C3, R8 to R10, R13 to R11, R14 to R12, R15 to R13, R16 to R14, R5 to R15, R6 to R16, R9 to R3, R3 to R4, R4 to R5, R10 to R6, R11 to R7, R7 to R8, R12 to R9, U3 to U1, U4 to U2, U5 to U3, U6 to U4, U7 to U5, U1 to U6
Connections:
- net Button_RCD39/To_MCP_PIN: now also U2.8 (GPB7)
- net FSR: now reaches R15.2, R16.1
Other:
- sheet Stm32f411retx ports: added FSR; removed none
- moved on the sheet: C2, R11, R15, R3, R6, R7, R9, U3, U5, U6

Commit message: added comments
Parts:
- removed U5: CP2102N-Axx-xQFN24, Package_DFN_QFN:QFN-24-1EP_4x4mm_P0.5mm_EP2.6x2.6mm, symbol Interface_USB:CP2102N-Axx-xQFN24
Other:
- note added: "J'ai relié les interruptions au stm32 mais j'ai un peu des doutes, je veux bien qu'on check si c'est ok"
- note added: "Pour le fsr je pense que je vais changer afin d'avoir une connectique avec des cables dupont (mettre du coup des connecteurs verticaux) J'aimerais bien faire un montage mécanique dans un second temps du coup il faudrait que je puisse mettre des cables un peu long afin de relier le fsr. Je souhaiterai aussi déporter un boutton poussoir voir plusieurs"
Changed lines of the file:
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@@
 	(generator_version "9.0")
 	(paper "A3")
+	(text "Pour le fsr je pense que je vais changer afin d'avoir une connectique\n avec des cables dupont (mettre du coup des connecteurs verticaux)\nJ'aimerais bien faire un montage mécanique dans un second temps \ndu coup il faudrait que je puisse mettre des cables un peu long\n afin de relier le fsr.\n\nJe souhaiterai aussi déporter un boutton poussoir voir plusieurs"
+		(exclude_from_sim no)
+		(at 210.566 207.772 0)
+		(effects
+			(font
+				(size 1.27 1.27)
+			)
+		)
+	)
+	(text "J'ai relié les interruptions au stm32 mais j'ai un peu des doutes, je veux bien qu'on check si c'est ok"
+		(exclude_from_sim no)
+		(at 77.724 16.764 0)
+		(effects
+			(font
+				(size 1.27 1.27)
+			)
+		)
+	)
 	(text_box "+ Passer tous les boitîer en version CMS :\n=> MCP23017 version SOIC \n=> Resistance, capa en CMS 0603\n+ Côté MCP23017 il faut câbler INTA et INTB et les pullup avec un 10K comme sure RESET (voir schéma adafruit)\n+ Précise les valeurs des composants aussi (comme j'ai fais sur la page bouton)\n+ Pour simplifier la lecture j'ai ajouté des labels je l'ai fais que côté I2C. On peut surement le faire ailleurs.\n+ J'ai du mal à ajouter d'autre pages au schematics. J'aimerai en créer une autre pour ajouter ton convertisseur de tension 5/3,3VDC (si on fais sauter blackpill)\n+ J'ai ajouté le MCU STM32F411RET6 et le convertisseur USB TTL histoire de faire sauter ton blackpill :p"
 		(exclude_from_sim no)
@@
 	(wire
 		(pts
-			(xy 111.76 236.22) (xy 119.38 236.22)
+			(xy 25.4 204.47) (xy 33.02 204.47)
 		)
 		(stroke
@@
 	(wire
 		(pts
-			(xy 119.38 246.38) (xy 110.49 246.38)
+			(xy 33.02 214.63) (xy 24.13 214.63)
 		)
 		(stroke
@@
 	(wire
 		(pts
-			(xy 110.49 254) (xy 119.38 254)
+			(xy 24.13 222.25) (xy 33.02 222.25)
 		)
 		(stroke
@@
 	(wire
 		(pts
-			(xy 133.35 224.79) (xy 133.35 229.87)
+			(xy 46.99 193.04) (xy 46.99 198.12)
 		)
 		(stroke
@@
 	(wire
 		(pts
-			(xy 111.76 232.41) (xy 119.38 232.41)
+			(xy 25.4 200.66) (xy 33.02 200.66)
 		)
 		(stroke
@@
 	(wire
 		(pts
-			(xy 111.76 238.76) (xy 119.38 238.76)
+			(xy 25.4 207.01) (xy 33.02 207.01)
 		)
 		(stroke
@@
 	(wire
 		(pts
-			(xy 119.38 250.19) (xy 110.49 250.19)
+			(xy 33.02 218.44) (xy 24.13 218.44)
 		)
 		(stroke
@@
 	(wire
 		(pts
-			(xy 137.16 238.76) (xy 142.24 238.76)
+			(xy 50.8 207.01) (xy 55.88 207.01)
 		)
 		(stroke
@@
 	(wire
 		(pts
-			(xy 137.16 243.84) (xy 142.24 243.84)
+			(xy 50.8 212.09) (xy 55.88 212.09)
 		)
 		(stroke
@@
 	(wire
 		(pts
-			(xy 110.49 259.08) (xy 119.38 259.08)
+			(xy 24.13 227.33) (xy 33.02 227.33)
 		)
 		(stroke
@@
 	)
 	(label "BCLCK"
-		(at 142.24 238.76 0)
+		(at 55.88 207.01 0)
 		(effects
 			(font
@@
 	)
 	(label "WSEL"
-		(at 133.35 224.79 0)
+		(at 46.99 193.04 0)
 		(effects
 			(font
@@
 	)
 	(label "SDA"
-		(at 111.76 236.22 0)
+		(at 25.4 204.47 0)
 		(effects
 			(font
@@
 	)
 	(label "FSR"
-		(at 142.24 243.84 0)
+		(at 55.88 212.09 0)
 		(effects
 			(font
@@
 	)
 	(label "INT4"
-		(at 110.49 259.08 0)
+		(at 24.13 227.33 0)
 		(effects
 			(font
@@
 	)
 	(label "SCL"
-		(at 111.76 232.41 0)
+		(at 25.4 200.66 0)
 		(effects
 			(font
@@
 	)
 	(label "INT1"
-		(at 110.49 246.38 0)
+		(at 24.13 214.63 0)
 		(effects
 			(font
@@
 	)
 	(label "INT3"
-		(at 110.49 254 0)
+		(at 24.13 222.25 0)
 		(effects
 			(font
@@
 	)
 	(label "INT2"
-		(at 110.49 250.19 0)
+		(at 24.13 218.44 0)
 		(effects
 			(font
@@
 	)
 	(label "MOSI"
-		(at 111.76 238.76 0)
+		(at 25.4 207.01 0)
 		(effects
 			(font
@@
 	)
 	(symbol
-		(lib_id "Interface_USB:CP2102N-Axx-xQFN24")
-		(at 60.96 246.38 0)
-		(unit 1)
-		(exclude_from_sim no)
-		(in_bom yes)
-		(on_board yes)
-		(dnp no)
-		(fields_autoplaced yes)
-		(property "Reference" "U5"
-			(at 63.1033 274.32 0)
-			(effects
-				(font
-					(size 1.27 1.27)
-				)
-				(justify left)
-			)
-		)
-		(property "Value" "CP2102N-Axx-xQFN24"
-			(at 63.1033 276.86 0)
-			(effects
-				(font
-					(size 1.27 1.27)
-				)
-				(justify left)
-			)
-		)
-		(property "Footprint" "Package_DFN_QFN:QFN-24-1EP_4x4mm_P0.5mm_EP2.6x2.6mm"
-			(at 92.71 273.05 0)
-			(effects
-				(font
-					(size 1.27 1.27)
-				)
-				(hide yes)
-			)
-		)
-		(property "Datasheet" "https://www.silabs.com/documents/public/data-sheets/cp2102n-datasheet.pdf"
-			(at 62.23 265.43 0)
-			(effects
-				(font
-					(size 1.27 1.27)
-				)
-				(hide yes)
-			)
-		)
-		(property "Description" "USB to UART master bridge, QFN-24"
-			(at 60.96 246.38 0)
-			(effects
-				(font
-					(size 1.27 1.27)
-				)
-				(hide yes)
-			)
-		)
-		(pin "9"
-		)
-		(pin "8"
-		)
-		(pin "11"
-		)
-		(pin "10"
-		)
-		(pin "7"
-		)
-		(pin "6"
-		)
-		(pin "2"
-		)
-		(pin "16"
-		)
-		(pin "3"
-		)
-		(pin "5"
-		)
-		(pin "17"
-		)
-		(pin "1"
-		)
-		(pin "24"
-		)
-		(pin "20"
-		)
-		(pin "23"
-		)
-		(pin "12"
-		)
-		(pin "19"
-		)
-		(pin "25"
-		)
-		(pin "4"
-		)
-		(pin "21"
-		)
-		(pin "22"
-		)
-		(pin "15"
-		)
-		(pin "14"
-		)
-		(pin "13"
-		)
-		(pin "18"
-		)
-		(instances
-			(project ""
-				(path "/2c0b0e0d-c5e7-48b7-93bb-9be1941509af"
-					(reference "U5")
-					(unit 1)
-				)
-			)
-		)
-	)
-	(symbol
 		(lib_id "power:+3.3V")
 		(at 331.47 36.83 0)
@@
 	)
 	(sheet
-		(at 119.38 229.87)
+		(at 33.02 198.12)
 		(size 17.78 34.29)
 		(exclude_from_sim no)
@@
 		)
 		(property "Sheetname" "Stm32f411retx"
-			(at 119.38 229.1584 0)
+			(at 33.02 197.4084 0)
 			(effects
 				(font
@@
 		)
 		(property "Sheetfile" "stm32f411retx.kicad_sch"
-			(at 119.38 264.7446 0)
+			(at 33.02 232.9946 0)
 			(effects
 				(font
@@
 		)
 		(pin "MOSI" input
-			(at 119.38 238.76 180)
+			(at 33.02 207.01 180)
 			(effects
 				(font
@@
 		)
 		(pin "MISO" input
-			(at 119.38 242.57 180)
+			(at 33.02 210.82 180)
 			(effects
 				(font
@@
 		)
 		(pin "INT1" output
-			(at 119.38 246.38 180)
+			(at 33.02 214.63 180)
 			(effects
 				(font
@@
 		)
 		(pin "INT2" output
-			(at 119.38 250.19 180)
+			(at 33.02 218.44 180)
 			(effects
 				(font
@@
 		)
 		(pin "INT3" output
-			(at 119.38 254 180)
+			(at 33.02 222.25 180)
 			(effects
 				(font
@@
 		)
 		(pin "INT4" output
-			(at 119.38 259.08 180)
+			(at 33.02 227.33 180)
 			(effects
 				(font
@@
 		)
 		(pin "SCL" bidirectional
-			(at 119.38 232.41 180)
+			(at 33.02 200.66 180)
 			(effects
 				(font
@@
 		)
 		(pin "SDA" bidirectional
-			(at 119.38 236.22 180)
+			(at 33.02 204.47 180)
 			(effects
 				(font
@@
 		)
 		(pin "WSEL" bidirectional
-			(at 133.35 229.87 90)
+			(at 46.99 198.12 90)
 			(effects
 				(font
@@
 		)
 		(pin "BCLCK" bidirectional
-			(at 137.16 238.76 0)
+			(at 50.8 207.01 0)
 			(effects
 				(font
@@
 		)
 		(pin "FSR" bidirectional
-			(at 137.16 243.84 0)
+			(at 50.8 212.09 0)
 			(effects
 				(font

Commit message: add values
Changed lines of the file:
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@@
 	)
 	(junction
-		(at 153.67 250.19)
+		(at 96.52 248.92)
 		(diameter 0)
 		(color 0 0 0 0)
@@
 	)
 	(junction
-		(at 172.72 250.19)
+		(at 115.57 248.92)
 		(diameter 0)
 		(color 0 0 0 0)
@@
 	(wire
 		(pts
-			(xy 172.72 250.19) (xy 170.18 250.19)
+			(xy 115.57 248.92) (xy 113.03 248.92)
 		)
 		(stroke
@@
 	(wire
 		(pts
-			(xy 153.67 250.19) (xy 153.67 251.46)
+			(xy 96.52 248.92) (xy 96.52 250.19)
 		)
 		(stroke
@@
 	(wire
 		(pts
-			(xy 175.26 250.19) (xy 172.72 250.19)
+			(xy 118.11 248.92) (xy 115.57 248.92)
 		)
 		(stroke
@@
 	(wire
 		(pts
-			(xy 157.48 250.19) (xy 153.67 250.19)
+			(xy 100.33 248.92) (xy 96.52 248.92)
 		)
 		(stroke
@@
 	(symbol
 		(lib_id "power:+3.3V")
-		(at 175.26 250.19 0)
+		(at 118.11 248.92 0)
 		(unit 1)
 		(exclude_from_sim no)
@@
 		(fields_autoplaced yes)
 		(property "Reference" "#PWR042"
-			(at 175.26 254 0)
+			(at 118.11 252.73 0)
 			(effects
 				(font
@@
 		)
 		(property "Value" "+3.3V"
-			(at 175.26 245.11 0)
+			(at 118.11 243.84 0)
 			(effects
 				(font
@@
 		)
 		(property "Footprint" ""
-			(at 175.26 250.19 0)
+			(at 118.11 248.92 0)
 			(effects
 				(font
@@
 		)
 		(property "Datasheet" ""
-			(at 175.26 250.19 0)
+			(at 118.11 248.92 0)
 			(effects
 				(font
@@
 		)
 		(property "Description" "Power symbol creates a global label with name \"+3.3V\""
-			(at 175.26 250.19 0)
+			(at 118.11 248.92 0)
 			(effects
 				(font
@@
 	(symbol
 		(lib_id "power:GND")
-		(at 153.67 250.19 0)
+		(at 96.52 248.92 0)
 		(unit 1)
 		(exclude_from_sim no)
@@
 		(fields_autoplaced yes)
 		(property "Reference" "#PWR041"
-			(at 153.67 256.54 0)
+			(at 96.52 255.27 0)
 			(effects
 				(font
@@
 		)
 		(property "Value" "GND"
-			(at 153.67 255.27 0)
+			(at 96.52 254 0)
 			(effects
 				(font
@@
 		)
 		(property "Footprint" ""
-			(at 153.67 250.19 0)
+			(at 96.52 248.92 0)
 			(effects
 				(font
@@
 		)
 		(property "Datasheet" ""
-			(at 153.67 250.19 0)
+			(at 96.52 248.92 0)
 			(effects
 				(font
@@
 		)
 		(property "Description" "Power symbol creates a global label with name \"GND\" , ground"
-			(at 153.67 250.19 0)
+			(at 96.52 248.92 0)
 			(effects
 				(font
@@
 	)
 	(sheet
-		(at 157.48 234.95)
+		(at 100.33 233.68)
 		(size 15.24 30.48)
 		(exclude_from_sim no)
@@
 		)
 		(property "Sheetname" "Buck"
-			(at 157.48 234.2384 0)
+			(at 100.33 232.9684 0)
 			(effects
 				(font
@@
 		)
 		(property "Sheetfile" "buck.kicad_sch"
-			(at 157.48 266.0146 0)
+			(at 100.33 264.7446 0)
 			(effects
 				(font
@@
 		)
 		(pin "3.3v" input
-			(at 172.72 250.19 0)
+			(at 115.57 248.92 0)
 			(effects
 				(font
@@
 		)
 		(pin "gnd" passive
-			(at 157.48 250.19 180)
+			(at 100.33 248.92 180)
 			(effects
 				(font
