File: kicadProjects/0511/0511/0511.kicad_sch (KiCad schematic)
At the start: 30 parts, among them U1 UDA1334A_Breakout

Commit message: début placement main gauche
Connections:
- net Button_RCD53/To_MCP_PIN is gone; now on an unnamed net: MCP23017_AD23.28 (GPA7)
- net at C5.1, R15.2, R16.1: no longer MCP23017_AD23.8 (GPB7)
- new net Button_RCD62/To_MCP_PIN: MCP23017_AD23.8 (GPB7)
Other:
- removed sheet Button_RCD53
- added sheet Button_RCD62 (buttonRcd.kicad_sch)
Changed lines of the file:
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@@
 	(wire
 		(pts
+			(xy 353.06 78.74) (xy 353.06 81.28)
+		)
+		(stroke
+			(width 0)
+			(type default)
+		)
+	)
+	(wire
+		(pts
 			(xy 152.4 96.52) (xy 152.4 99.06)
 		)
@@
 	(wire
 		(pts
-			(xy 353.06 144.78) (xy 367.03 144.78)
-		)
-		(stroke
-			(width 0)
-			(type default)
-		)
-	)
-	(wire
-		(pts
 			(xy 416.56 148.59) (xy 416.56 152.4)
 		)
@@
 	(wire
 		(pts
-			(xy 353.06 78.74) (xy 353.06 144.78)
-		)
-		(stroke
-			(width 0)
-			(type default)
-		)
-	)
-	(wire
-		(pts
 			(xy 207.01 243.84) (xy 213.36 243.84)
 		)
@@
 	(wire
 		(pts
+			(xy 331.47 78.74) (xy 331.47 144.78)
+		)
+		(stroke
+			(width 0)
+			(type default)
+		)
+	)
+	(wire
+		(pts
 			(xy 119.38 196.85) (xy 119.38 194.31)
 		)
@@
 	(wire
 		(pts
-			(xy 60.96 106.68) (xy 60.96 110.49)
+			(xy 331.47 144.78) (xy 367.03 144.78)
 		)
 		(stroke
@@
 	(wire
 		(pts
-			(xy 64.77 114.3) (xy 64.77 106.68)
+			(xy 60.96 106.68) (xy 60.96 110.49)
 		)
 		(stroke
@@
 	(wire
 		(pts
-			(xy 331.47 78.74) (xy 331.47 139.7)
+			(xy 64.77 114.3) (xy 64.77 106.68)
 		)
 		(stroke
@@
 	)
 	(sheet
-		(at 326.39 139.7)
+		(at 213.36 138.43)
 		(size 12.7 3.81)
 		(exclude_from_sim no)
@@
 			(color 0 0 0 0.0000)
 		)
-		(property "Sheetname" "Button_RCD53"
-			(at 326.39 138.9884 0)
+		(property "Sheetname" "Button_RCD83"
+			(at 213.36 137.7184 0)
 			(do_not_autoplace yes)
 			(effects
@@
 		)
 		(property "Sheetfile" "buttonRcd.kicad_sch"
-			(at 326.39 144.0946 0)
+			(at 213.36 142.8246 0)
 			(effects
 				(font
@@
 		)
 		(pin "To_MCP_PIN" input
-			(at 331.47 139.7 90)
+			(at 218.44 138.43 90)
 			(effects
 				(font
@@
 			(project "0511"
 				(path "/2c0b0e0d-c5e7-48b7-93bb-9be1941509af"
-					(page "56")
+					(page "48")
 				)
 			)
@@
 	)
 	(sheet
-		(at 213.36 138.43)
+		(at 115.57 161.29)
 		(size 12.7 3.81)
 		(exclude_from_sim no)
@@
 			(color 0 0 0 0.0000)
 		)
-		(property "Sheetname" "Button_RCD83"
-			(at 213.36 137.7184 0)
+		(property "Sheetname" "Button_RCD22"
+			(at 115.57 160.5784 0)
 			(do_not_autoplace yes)
 			(effects
@@
 		)
 		(property "Sheetfile" "buttonRcd.kicad_sch"
-			(at 213.36 142.8246 0)
+			(at 115.57 165.6846 0)
 			(effects
 				(font
@@
 		)
 		(pin "To_MCP_PIN" input
-			(at 218.44 138.43 90)
+			(at 120.65 161.29 90)
 			(effects
 				(font
@@
 			(project "0511"
 				(path "/2c0b0e0d-c5e7-48b7-93bb-9be1941509af"
-					(page "48")
+					(page "24")
 				)
 			)
@@
 	)
 	(sheet
-		(at 115.57 161.29)
+		(at 347.98 81.28)
 		(size 12.7 3.81)
 		(exclude_from_sim no)
@@
 			(color 0 0 0 0.0000)
 		)
-		(property "Sheetname" "Button_RCD22"
-			(at 115.57 160.5784 0)
-			(do_not_autoplace yes)
+		(property "Sheetname" "Button_RCD62"
+			(at 347.98 80.5684 0)
 			(effects
 				(font
@@
 		)
 		(property "Sheetfile" "buttonRcd.kicad_sch"
-			(at 115.57 165.6846 0)
+			(at 347.98 85.6746 0)
 			(effects
 				(font
@@
 		)
 		(pin "To_MCP_PIN" input
-			(at 120.65 161.29 90)
+			(at 353.06 81.28 90)
 			(effects
 				(font
@@
 			(project "0511"
 				(path "/2c0b0e0d-c5e7-48b7-93bb-9be1941509af"
-					(page "24")
+					(page "4")
 				)
 			)

Commit message: added B port interruptions, updated schem and pcb
Connections:
- net INTB4: now reaches MCP23017_AD23.19 (INTB), PULLUP_INTB_23.2
- net INTB3: now reaches MCP23017_ADD22.19 (INTB), PULLUP_INTB_22.2
- net INTB2: now reaches MCP23017_ADD21.19 (INTB), PULLUP_INTB_21.2
- net INTB1: now reaches MCP23017_ADD20.19 (INTB), PULLUP_INTB_20.2
Other:
- sheet Stm32f411retx ports: added INTB1, INTB2, INTB3, INTB4; removed none

Commit message: correctif adafruit component
Connections:
- net +3.3V: now also U1.5 (3V); no longer U1.1 (VIN)
- net BCLCK: now also U1.1 (BCLK); no longer U1.5 (BCLK)
- net GND: now also U1.4 (GND); no longer U1.3 (GND)
- net MOSI: now also U1.2 (DIN); no longer U1.6 (DIN)
- net WSEL: now also U1.3 (WSEL); no longer U1.4 (WSEL)
Other:
- sheet Stm32f411retx ports: added none; removed MISO
Changed lines of the file:
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@@
 	)
 	(junction
+		(at 260.35 250.19)
+		(diameter 0)
+		(color 0 0 0 0)
+	)
+	(junction
 		(at 152.4 107.95)
 		(diameter 0)
@@
 	(wire
 		(pts
-			(xy 260.35 248.92) (xy 251.46 248.92)
+			(xy 353.06 78.74) (xy 353.06 81.28)
 		)
 		(stroke
@@
 	(wire
 		(pts
-			(xy 353.06 78.74) (xy 353.06 81.28)
+			(xy 152.4 96.52) (xy 152.4 99.06)
 		)
 		(stroke
@@
 	(wire
 		(pts
-			(xy 152.4 96.52) (xy 152.4 99.06)
+			(xy 59.69 106.68) (xy 58.42 106.68)
 		)
 		(stroke
@@
 	(wire
 		(pts
-			(xy 59.69 106.68) (xy 58.42 106.68)
+			(xy 114.3 113.03) (xy 114.3 115.57)
 		)
 		(stroke
@@
 	(wire
 		(pts
-			(xy 114.3 113.03) (xy 114.3 115.57)
+			(xy 260.35 245.11) (xy 243.84 245.11)
 		)
 		(stroke
@@
 	(wire
 		(pts
+			(xy 247.65 252.73) (xy 260.35 252.73)
+		)
+		(stroke
+			(width 0)
+			(type default)
+		)
+	)
+	(wire
+		(pts
 			(xy 134.62 104.14) (xy 134.62 107.95)
 		)
@@
 	(wire
 		(pts
-			(xy 247.65 242.57) (xy 247.65 245.11)
-		)
-		(stroke
-			(width 0)
-			(type default)
-		)
-	)
-	(wire
-		(pts
 			(xy 372.11 36.83) (xy 372.11 43.18)
 		)
@@
 	(wire
 		(pts
-			(xy 251.46 248.92) (xy 251.46 247.65)
+			(xy 274.32 105.41) (xy 274.32 111.76)
 		)
 		(stroke
@@
 	(wire
 		(pts
-			(xy 274.32 105.41) (xy 274.32 111.76)
+			(xy 238.76 247.65) (xy 260.35 247.65)
 		)
 		(stroke
@@
 	(wire
 		(pts
+			(xy 257.81 255.27) (xy 260.35 255.27)
+		)
+		(stroke
+			(width 0)
+			(type default)
+		)
+	)
+	(wire
+		(pts
 			(xy 367.03 144.78) (xy 367.03 127)
 		)
@@
 	(wire
 		(pts
+			(xy 257.81 255.27) (xy 257.81 257.81)
+		)
+		(stroke
+			(width 0)
+			(type default)
+		)
+	)
+	(wire
+		(pts
 			(xy 358.14 78.74) (xy 356.87 78.74)
 		)
@@
 	(wire
 		(pts
-			(xy 242.57 252.73) (xy 260.35 252.73)
-		)
-		(stroke
-			(width 0)
-			(type default)
-		)
-	)
-	(wire
-		(pts
 			(xy 167.64 156.21) (xy 172.72 156.21)
 		)
@@
 	(wire
 		(pts
-			(xy 250.19 247.65) (xy 250.19 248.92)
-		)
-		(stroke
-			(width 0)
-			(type default)
-		)
-	)
-	(wire
-		(pts
 			(xy 275.59 120.65) (xy 275.59 118.11)
 		)
@@
 	(wire
 		(pts
-			(xy 242.57 255.27) (xy 260.35 255.27)
-		)
-		(stroke
-			(width 0)
-			(type default)
-		)
-	)
-	(wire
-		(pts
 			(xy 255.27 105.41) (xy 254 105.41)
 		)
@@
 	(wire
 		(pts
-			(xy 275.59 247.65) (xy 275.59 251.46)
-		)
-		(stroke
-			(width 0)
-			(type default)
-		)
-	)
-	(wire
-		(pts
 			(xy 342.9 115.57) (xy 342.9 120.65)
 		)
@@
 	(wire
 		(pts
+			(xy 243.84 250.19) (xy 260.35 250.19)
+		)
+		(stroke
+			(width 0)
+			(type default)
+		)
+	)
+	(wire
+		(pts
 			(xy 217.17 77.47) (xy 217.17 80.01)
 		)
@@
 	(wire
 		(pts
-			(xy 260.35 245.11) (xy 247.65 245.11)
-		)
-		(stroke
-			(width 0)
-			(type default)
-		)
-	)
-	(wire
-		(pts
 			(xy 228.6 63.5) (xy 228.6 69.85)
 		)
@@
 	(wire
 		(pts
-			(xy 281.94 251.46) (xy 275.59 251.46)
-		)
-		(stroke
-			(width 0)
-			(type default)
-		)
-	)
-	(wire
-		(pts
 			(xy 134.62 143.51) (xy 134.62 185.42)
 		)
@@
 	(wire
 		(pts
-			(xy 64.77 114.3) (xy 64.77 106.68)
+			(xy 243.84 245.11) (xy 243.84 246.38)
 		)
 		(stroke
@@
 	(wire
 		(pts
-			(xy 308.61 105.41) (xy 344.17 105.41)
+			(xy 64.77 114.3) (xy 64.77 106.68)
 		)
 		(stroke
@@
 	(wire
 		(pts
-			(xy 218.44 128.27) (xy 243.84 128.27)
+			(xy 308.61 105.41) (xy 344.17 105.41)
 		)
 		(stroke
@@
 	(wire
 		(pts
-			(xy 311.15 120.65) (xy 336.55 120.65)
+			(xy 218.44 128.27) (xy 243.84 128.27)
 		)
 		(stroke
@@
 	(wire
 		(pts
-			(xy 22.86 133.35) (xy 45.72 133.35)
+			(xy 311.15 120.65) (xy 336.55 120.65)
 		)
 		(stroke
@@
 	(wire
 		(pts
-			(xy 205.74 147.32) (xy 205.74 151.13)
+			(xy 22.86 133.35) (xy 45.72 133.35)
 		)
 		(stroke
@@
 	(wire
 		(pts
-			(xy 411.48 152.4) (xy 416.56 152.4)
+			(xy 205.74 147.32) (xy 205.74 151.13)
 		)
 		(stroke
@@
 	(wire
 		(pts
-			(xy 377.19 78.74) (xy 377.19 85.09)
+			(xy 411.48 152.4) (xy 416.56 152.4)
 		)
 		(stroke
@@
 	(wire
 		(pts
-			(xy 251.46 247.65) (xy 250.19 247.65)
+			(xy 377.19 78.74) (xy 377.19 85.09)
 		)
 		(stroke
@@
 	)
 	(label "BCLCK"
-		(at 242.57 255.27 0)
+		(at 243.84 246.38 0)
 		(effects
 			(font
@@
 	)
 	(label "MOSI"
-		(at 281.94 251.46 0)
+		(at 238.76 247.65 0)
 		(effects
 			(font
@@
 	)
 	(label "WSEL"
-		(at 242.57 252.73 0)
+		(at 243.84 250.19 0)
 		(effects
 			(font
@@
 	(symbol
 		(lib_id "power:+3.3V")
-		(at 247.65 242.57 0)
+		(at 257.81 257.81 180)
 		(unit 1)
 		(exclude_from_sim no)
@@
 		(fields_autoplaced yes)
 		(property "Reference" "#PWR041"
-			(at 247.65 246.38 0)
+			(at 257.81 254 0)
 			(effects
 				(font
@@
 		)
 		(property "Value" "+3.3V"
-			(at 247.65 237.49 0)
+			(at 257.81 262.89 0)
 			(effects
 				(font
@@
 		)
 		(property "Footprint" ""
-			(at 247.65 242.57 0)
+			(at 257.81 257.81 0)
 			(effects
 				(font
@@
 		)
 		(property "Datasheet" ""
-			(at 247.65 242.57 0)
+			(at 257.81 257.81 0)
 			(effects
 				(font
@@
 		)
 		(property "Description" "Power symbol creates a global label with name \"+3.3V\""
-			(at 247.65 242.57 0)
+			(at 257.81 257.81 0)
 			(effects
 				(font
@@
 	(symbol
 		(lib_id "power:GND")
-		(at 250.19 248.92 0)
+		(at 247.65 252.73 0)
 		(unit 1)
 		(exclude_from_sim no)
@@
 		(fields_autoplaced yes)
 		(property "Reference" "#PWR042"
-			(at 250.19 255.27 0)
+			(at 247.65 259.08 0)
 			(effects
 				(font
@@
 		)
 		(property "Value" "GND"
-			(at 250.19 254 0)
+			(at 247.65 257.81 0)
 			(effects
 				(font
@@
 		)
 		(property "Footprint" ""
-			(at 250.19 248.92 0)
+			(at 247.65 252.73 0)
 			(effects
 				(font
@@
 		)
 		(property "Datasheet" ""
-			(at 250.19 248.92 0)
+			(at 247.65 252.73 0)
 			(effects
 				(font
@@
 		)
 		(property "Description" "Power symbol creates a global label with name \"GND\" , ground"
-			(at 250.19 248.92 0)
+			(at 247.65 252.73 0)
 			(effects
 				(font
@@
 			(effects
 				(font
-					(size 1.27 1.27)
-				)
-				(justify left)
-			)
-		)
-		(pin "MISO" input
-			(at 33.02 210.82 180)
-			(effects
-				(font

Commit message: correctif empreinte, ajout tests points
Connections:
- net +3.3V: now also U1.9 (VIN); no longer U1.5 (3V)
- net BCLCK: now also U1.4 (BCLK); no longer U1.1 (BCLK)
- net GND: now also U1.7 (GND); no longer U1.4 (GND)
- net MOSI: now also U1.5 (DIN); no longer U1.2 (DIN)
- net WSEL: now also U1.6 (WSEL); no longer U1.3 (WSEL)
Changed lines of the file:
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@@
 	(wire
 		(pts
-			(xy 257.81 255.27) (xy 257.81 257.81)
-		)
-		(stroke
-			(width 0)
-			(type default)
-		)
-	)
-	(wire
-		(pts
 			(xy 358.14 78.74) (xy 356.87 78.74)
 		)
@@
 	(wire
 		(pts
+			(xy 275.59 247.65) (xy 275.59 251.46)
+		)
+		(stroke
+			(width 0)
+			(type default)
+		)
+	)
+	(wire
+		(pts
 			(xy 217.17 87.63) (xy 217.17 88.9)
 		)
@@
 			)
 		)
-		(pin "2"
+		(pin "8"
 		)
-		(pin "1"
+		(pin "7"
 		)
-		(pin "3"
+		(pin "9"
 		)
 		(pin "5"
@@
 	(symbol
 		(lib_id "power:+3.3V")
-		(at 257.81 257.81 180)
+		(at 275.59 251.46 180)
 		(unit 1)
 		(exclude_from_sim no)
@@
 		(fields_autoplaced yes)
 		(property "Reference" "#PWR041"
-			(at 257.81 254 0)
+			(at 275.59 247.65 0)
 			(effects
 				(font
@@
 		)
 		(property "Value" "+3.3V"
-			(at 257.81 262.89 0)
+			(at 275.59 256.54 0)
 			(effects
 				(font
@@
 		)
 		(property "Footprint" ""
-			(at 257.81 257.81 0)
+			(at 275.59 251.46 0)
 			(effects
 				(font
@@
 		)
 		(property "Datasheet" ""
-			(at 257.81 257.81 0)
+			(at 275.59 251.46 0)
 			(effects
 				(font
@@
 		)
 		(property "Description" "Power symbol creates a global label with name \"+3.3V\""
-			(at 257.81 257.81 0)
+			(at 275.59 251.46 0)
 			(effects
 				(font

Commit message: correction, début mise en place BOM
Parts:
- R17: value ~ -> 10K
- R6: value 4,7k -> 4,7K
Changed lines of the file:
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@@
 			)
 		)
-		(property "Value" "4,7k"
+		(property "Value" "4,7K"
 			(at 62.992 53.594 0)
 			(effects
@@
 			)
 		)
-		(property "Value" "~"
+		(property "Value" "10K"
 			(at 209.55 250.1899 0)
 			(effects

Commit message: correctifs valeurs manquantes
Parts:
- A7_23_C1: renamed from C5; value 1uF -> 100nF
- renumbered D1 to A7_23_D1, R16 to A7_23_R1, R15 to A7_23_R2
Changed lines of the file:
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@@
 		(dnp no)
 		(fields_autoplaced yes)
-		(property "Reference" "R16"
+		(property "Reference" "A7_23_R1"
 			(at 407.67 146.05 90)
 			(effects
@@
 			(project "0511"
 				(path "/2c0b0e0d-c5e7-48b7-93bb-9be1941509af"
-					(reference "R16")
+					(reference "A7_23_R1")
 					(unit 1)
 				)
@@
 		(dnp no)
 		(fields_autoplaced yes)
-		(property "Reference" "D1"
+		(property "Reference" "A7_23_D1"
 			(at 394.6525 146.05 0)
 			(effects
@@
 			(project "0511"
 				(path "/2c0b0e0d-c5e7-48b7-93bb-9be1941509af"
-					(reference "D1")
+					(reference "A7_23_D1")
 					(unit 1)
 				)
@@
 		(dnp no)
 		(fields_autoplaced yes)
-		(property "Reference" "C5"
+		(property "Reference" "A7_23_C1"
 			(at 420.37 157.4799 0)
 			(effects
@@
 			)
 		)
-		(property "Value" "1uF"
+		(property "Value" "100nF"
 			(at 420.37 160.0199 0)
 			(effects
@@
 			(project "0511"
 				(path "/2c0b0e0d-c5e7-48b7-93bb-9be1941509af"
-					(reference "C5")
+					(reference "A7_23_C1")
 					(unit 1)
 				)
@@
 		(dnp no)
 		(fields_autoplaced yes)
-		(property "Reference" "R15"
+		(property "Reference" "A7_23_R2"
 			(at 419.1 143.5099 0)
 			(effects
@@
 			(project "0511"
 				(path "/2c0b0e0d-c5e7-48b7-93bb-9be1941509af"
-					(reference "R15")
-					(unit 1)
-				)
+					(reference "A7_23_R2")
+					(unit 1)
+				)

Commit message: ajout dossier fabrication
Parts:
- R17: value 10K -> 22K
Changed lines of the file:
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@@
 			)
 		)
-		(property "Value" "10K"
+		(property "Value" "22K"
 			(at 209.55 250.1899 0)
 			(effects
