File: kicadProjects/0511/0511/buck.kicad_sch (KiCad schematic)
At the start: 9 parts, among them U9 LM2575-3.3BT

Commit message: assignation empreintes
Parts:
- C72, C73: footprint (none) -> Capacitor_Tantalum_SMD:CP_EIA-6032-28_Kemet-C
- D69: footprint (none) -> LED_SMD:LED_0603_1608Metric
- L1: footprint (none) -> Inductor_SMD:L_0603_1608Metric
- R151, R152, R153: footprint (none) -> Resistor_SMD:R_0603_1608Metric
- renumbered U9 to U7
Changed lines of the file:
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@@
 			)
 		)
-		(property "Footprint" ""
+		(property "Footprint" "Resistor_SMD:R_0603_1608Metric"
 			(at 116.332 44.45 90)
 			(effects
@@
 			)
 		)
-		(property "Footprint" ""
+		(property "Footprint" "Inductor_SMD:L_0603_1608Metric"
 			(at 82.55 38.1 0)
 			(effects
@@
 			)
 		)
-		(property "Footprint" ""
+		(property "Footprint" "Capacitor_Tantalum_SMD:CP_EIA-6032-28_Kemet-C"
 			(at 23.8252 45.72 0)
 			(effects
@@
 			)
 		)
-		(property "Footprint" ""
+		(property "Footprint" "Capacitor_Tantalum_SMD:CP_EIA-6032-28_Kemet-C"
 			(at 100.0252 49.53 0)
 			(effects
@@
 			)
 		)
-		(property "Footprint" ""
+		(property "Footprint" "Resistor_SMD:R_0603_1608Metric"
 			(at 116.332 54.61 90)
 			(effects
@@
 		(dnp no)
 		(fields_autoplaced yes)
-		(property "Reference" "U9"
+		(property "Reference" "U7"
 			(at 60.96 25.4 0)
 			(effects
@@
 			(project ""
 				(path "/2c0b0e0d-c5e7-48b7-93bb-9be1941509af/88fc5341-afb8-4308-b309-3807a8feeae9"
-					(reference "U9")
+					(reference "U7")
 					(unit 1)
 				)
@@
 		(dnp no)
 		(fields_autoplaced yes)
-		(property "Reference" "#PWR0180"
+		(property "Reference" "#PWR0178"
 			(at 33.02 31.75 0)
 			(effects
@@
 			(project ""
 				(path "/2c0b0e0d-c5e7-48b7-93bb-9be1941509af/88fc5341-afb8-4308-b309-3807a8feeae9"
-					(reference "#PWR0180")
+					(reference "#PWR0178")
 					(unit 1)
 				)
@@
 			)
 		)
-		(property "Footprint" ""
+		(property "Footprint" "Resistor_SMD:R_0603_1608Metric"
 			(at 131.572 44.45 90)
 			(effects
@@
 		(dnp no)
 		(fields_autoplaced yes)
-		(property "Reference" "#PWR0181"
+		(property "Reference" "#PWR0179"
 			(at 36.83 72.39 0)
 			(effects
@@
 			(project ""
 				(path "/2c0b0e0d-c5e7-48b7-93bb-9be1941509af/88fc5341-afb8-4308-b309-3807a8feeae9"
-					(reference "#PWR0181")
+					(reference "#PWR0179")
 					(unit 1)
 				)
@@
 			)
 		)
-		(property "Footprint" ""
+		(property "Footprint" "LED_SMD:LED_0603_1608Metric"
 			(at 133.35 54.61 0)
 			(effects

Commit message: added comments
Other:
- note added: "J'ai pas mis les valeurs de composants pour le moment J'ai des doutes sur les empreintes"
Changed lines of the file:
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@@
 	(generator_version "9.0")
 	(paper "A4")
+	(text "J'ai pas mis les valeurs de composants pour le moment \n\nJ'ai des doutes sur les empreintes"
+		(exclude_from_sim no)
+		(at 221.234 174.498 0)
+		(effects
+			(font
+				(size 1.27 1.27)
+			)
+		)
+	)
 	(junction
 		(at 36.83 59.69)

Commit message: add values
Parts:
- C72: value C_Polarized -> EEEP1V221AP_AJUSTER_EMPREINTE
Changed lines of the file:
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@@
 			)
 		)
-		(property "Value" "C_Polarized"
+		(property "Value" "EEEP1V221AP_AJUSTER_EMPREINTE"
 			(at 26.67 42.2909 0)
 			(effects
