File: kicadProjects/0511/0511/_autosave-0511.kicad_pcb (KiCad board)
At the start: 2 copper layers, 527.5 x 359.5 mm, 377 parts, among them J1 USB4120-03-C_REVA6, U5 UDA1334A_Breakout, U6 STM32F411RETx, U7 BD33HC5WEFJ-E2, Y1 32.768KHz, Y2 8MHz

Commit message: poursuite placement et nommage références
Parts:
- renumbered A0_20 to A0_1, A0_21 to A0_2, C11 to A0_20_C1, D7 to A0_20_D1, R28 to A0_20_R1, R29 to A0_20_R2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
