File: kicadProjects/0511/0511/_autosave-stm32f411retx.kicad_sch (KiCad schematic)
At the start: 21 parts, among them U2 STM32F411RETx, Y1 32.768KHz, Y2 8MHz

Commit message: ajouut ferrite
Parts:
- gave numbers to parts that had none: 2
Changed lines of the file:
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@@
 		(dnp no)
 		(fields_autoplaced yes)
-		(property "Reference" "FB?"
+		(property "Reference" "FB1"
 			(at 88.9 139.6491 0)
 			(effects
@@
 			(project ""
 				(path "/2c0b0e0d-c5e7-48b7-93bb-9be1941509af/7f025c79-ea20-4013-a71e-871359ae3c80"
-					(reference "FB?")
+					(reference "FB1")
 					(unit 1)
 				)
@@
 		(on_board yes)
 		(dnp no)
-		(property "Reference" "C?"
+		(property "Reference" "C1"
 			(at 66.802 134.366 0)
 			(effects
@@
 			(project "0511"
 				(path "/2c0b0e0d-c5e7-48b7-93bb-9be1941509af/7f025c79-ea20-4013-a71e-871359ae3c80"
-					(reference "C?")
-					(unit 1)
-				)
+					(reference "C1")
+					(unit 1)
+				)
