File: kicadProjects/0511/0511/buttonRcd.kicad_sch (KiCad schematic)
At the start: 5 parts

Commit message: poursuite annotaion circuits rdc
Parts:
- renumbered A6_1 to A6_20, C6 to A6_20_C1, D2 to A6_20_D1, R19 to A6_20_R1, R18 to A6_20_R2

Commit message: corrected DRC errors
Parts:
- A6_20_C1: value 1uF -> 100nF
Changed lines of the file:
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@@
 			)
 		)
-		(property "Value" "1uF"
+		(property "Value" "100nF"
 			(at 180.34 110.4899 0)
 			(effects
