File: kicadProjects/0511/0511/usbc.kicad_sch (KiCad schematic)
At the start: 13 parts, among them J1 USB4120-03-C_REVA6, U3 BD33HC5WEFJ-E2

Commit message: correctifs valeurs manquantes
Parts:
- renumbered C75 to VBUS_C1
Connections:
- net 3.3V: now also U3.2 (VO_S)
Changed lines of the file:
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@@
+	)
+	(junction
+		(at 67.31 35.56)
+		(diameter 0)
+		(color 0 0 0 0)
 	)
 	(junction
@@
 	(wire
 		(pts
+			(xy 67.31 38.1) (xy 67.31 35.56)
+		)
+		(stroke
+			(width 0)
+			(type default)
+		)
+	)
+	(wire
+		(pts
 			(xy 67.31 40.64) (xy 57.15 40.64)
 		)
@@
 	(wire
 		(pts
-			(xy 67.31 35.56) (xy 52.07 35.56)
+			(xy 52.07 35.56) (xy 67.31 35.56)
 		)
 		(stroke
@@
 		(dnp no)
 		(property "Reference" "C73"
-			(at 131.826 43.688 90)
+			(at 132.08 43.942 90)
 			(effects
 				(font
@@
 		(on_board yes)
 		(dnp no)
-		(property "Reference" "C75"
+		(property "Reference" "VBUS_C1"
 			(at 74.676 88.138 90)
 			(effects
@@
 			(project "0511"
 				(path "/2c0b0e0d-c5e7-48b7-93bb-9be1941509af/7f025c79-ea20-4013-a71e-871359ae3c80/be8e2f48-706b-43bd-b6e8-a7bcf8b61384"
-					(reference "C75")
+					(reference "VBUS_C1")
 					(unit 1)
 				)
